File: hardware/MIRA_Control/400_MCU_RESERVED_GPIO.kicad_sch (KiCad schematic)
At the start: 1 part, among them U4101 STM32H745IIT6

Commit message: Save MIRA Control and Power baseline before PCB preparation
Parts:
- removed U4101: STM32H745IIT6, MIRA_RevA:LQFP-176_24x24mm_P0.5mm, symbol MIRA_RevA:STM32H745IIT6_MIRA
Connections:
- no-connect marks 49 -> 0
