File: hardware/MIRA_Control/500_MCU_SDRAM_64MB.kicad_sch (KiCad schematic)
At the start: 34 parts, among them U4501 IS42S16320F-7TLI

Commit message: Save MIRA Control and Power baseline before PCB preparation
Parts:
- removed C4501, C4502, C4503, C4504, C4505, C4506, C4507: 100n, MIRA_RevA:C_0201_0603Metric, symbol MIRA_RevA:Capacitor
- removed C4508: 4.7u, MIRA_RevA:C_0603_1608Metric, symbol MIRA_RevA:Capacitor
- removed R4501, R4502, R4503, R4504, R4505, R4506, R4507, R4508, R4509, R4510, R4511, R4512, R4513, R4514, R4515, R4516, R4517, R4518, R4519, R4520, R4521, R4522: 22, MIRA_RevA:R_0201_0603Metric, symbol MIRA_RevA:Resistor
- removed R4523: 33, MIRA_RevA:R_0201_0603Metric, symbol MIRA_RevA:Resistor
- removed R4524, R4525: 10k, MIRA_RevA:R_0201_0603Metric, symbol MIRA_RevA:Resistor
- removed U4501: IS42S16320F-7TLI, MIRA_RevA:TSOP-II-54_22.2x10.16mm_P0.8mm, symbol MIRA_RevA:IS42S16320F_7TLI_MIRA
Connections:
- no-connect marks 1 -> 0
Other:
- note removed: "4500_MCU_SDRAM_64MB"
- note removed: "Main MCU 64 MiB SDRAM | Rev.A"
- note removed: "Main MCU SDRAM source damping | Rev.A"
- note removed: "SDRAM supply bypass and reservoir"
