File: hardware/MIRA_Control/600_MCU_QSPI_FLASH.kicad_sch (KiCad schematic)
At the start: 12 parts, among them U4601 W25Q512JVEIQ

Commit message: Save MIRA Control and Power baseline before PCB preparation
Parts:
- removed C4601: 100n, MIRA_RevA:C_0201_0603Metric, symbol MIRA_RevA:Capacitor
- removed C4602: 1u, MIRA_RevA:C_0402_1005Metric, symbol MIRA_RevA:Capacitor
- removed R4601, R4602, R4603, R4604, R4605, R4606: 33, MIRA_RevA:R_0201_0603Metric, symbol MIRA_RevA:Resistor
- removed R4607, R4608, R4609: 10k, MIRA_RevA:R_0201_0603Metric, symbol MIRA_RevA:Resistor
- removed U4601: W25Q512JVEIQ, MIRA_RevA:WSON-8-1EP_8x6mm_P1.27mm_EP3.4x4.3mm, symbol MIRA_RevA:W25Q512JVEIQ_MIRA
Other:
- note removed: "4600_MCU_QSPI_FLASH"
- note removed: "Main MCU 64 MiB QSPI NOR flash | Rev.A"
