File: hardware/MIRA_Control/700_MCU_MICROSD.kicad_sch (KiCad schematic)
At the start: 18 parts, among them J4701 DM3AT-SF-PEJM5, U4701 USBLC6-2SC6, U4702 USBLC6-2SC6, U4703 USBLC6-2SC6

Commit message: Save MIRA Control and Power baseline before PCB preparation
Parts:
- removed C4701: 100n, MIRA_RevA:C_0201_0603Metric, symbol MIRA_RevA:Capacitor
- removed C4702: 10u, MIRA_RevA:C_0603_1608Metric, symbol MIRA_RevA:Capacitor
- removed J4701: DM3AT-SF-PEJM5, MIRA_RevA:microSD_HC_Hirose_DM3AT-SF-PEJM5, symbol MIRA_RevA:DM3AT_SF_PEJM5_MIRA
- removed R4701, R4702, R4703, R4704, R4705, R4706: 33, MIRA_RevA:R_0201_0603Metric, symbol MIRA_RevA:Resistor
- removed R4707, R4708, R4709, R4710, R4711: 47k, MIRA_RevA:R_0201_0603Metric, symbol MIRA_RevA:Resistor
- removed R4712: 10k, MIRA_RevA:R_0201_0603Metric, symbol MIRA_RevA:Resistor
- removed U4701, U4702, U4703: USBLC6-2SC6, MIRA_RevA:SOT-23-6, symbol MIRA_RevA:USBLC6_2SC6_MIRA
Other:
- note removed: "Main MCU microSD bias and ESD | Rev.A"
- note removed: "Main MCU microSD connector | Rev.A"
