File: hardware/MIRA_Control/800_MCU_CLOCK_RESET_DEBUG.kicad_sch (KiCad schematic)
At the start: 16 parts, among them J4801 Cortex SWD 10-pin, J4802 Boot jumper, SW4801 Reset pushbutton, U4101 STM32H745IIT6, Y4801 ASV-25.000MHZ-EJ-T, Y4802 ABS07-32.768KHZ-7-T

Commit message: Save MIRA Control and Power baseline before PCB preparation
Parts:
- removed C4801, C4804: 100n, MIRA_RevA:C_0201_0603Metric, symbol MIRA_RevA:Capacitor
- removed C4802, C4803: 12p, MIRA_RevA:C_0201_0603Metric, symbol MIRA_RevA:Capacitor
- removed J4801: Cortex SWD 10-pin, MIRA_RevA:PinHeader_2x05_P1.27mm_Vertical, symbol MIRA_RevA:Cortex_SWD_10_pin_MIRA
- removed J4802: Boot jumper, MIRA_RevA:PinHeader_1x02_P2.54mm_Vertical, symbol MIRA_RevA:Boot_jumper_MIRA
- removed R4801, R4803, R4804: 33, MIRA_RevA:R_0201_0603Metric, symbol MIRA_RevA:Resistor
- removed R4802, R4806: 10k, MIRA_RevA:R_0201_0603Metric, symbol MIRA_RevA:Resistor
- removed R4805: 100k, MIRA_RevA:R_0201_0603Metric, symbol MIRA_RevA:Resistor
- removed SW4801: Reset pushbutton, MIRA_RevA:SW_SPST_TL3342, symbol MIRA_RevA:Reset_pushbutton_MIRA
- removed U4101: STM32H745IIT6, MIRA_RevA:LQFP-176_24x24mm_P0.5mm, symbol MIRA_RevA:STM32H745IIT6_MIRA
- removed Y4801: ASV-25.000MHZ-EJ-T, MIRA_RevA:Oscillator_SMD_Abracon_ASV-4Pin_7.0x5.1mm, symbol MIRA_RevA:ASV_25_000MHZ_EJ_T_MIRA
- removed Y4802: ABS07-32.768KHZ-7-T, MIRA_RevA:Crystal_SMD_3215-2Pin_3.2x1.5mm, symbol MIRA_RevA:ABS07_32_768KHZ_7_T_MIRA
Connections:
- no-connect marks 3 -> 0
Other:
- note removed: "Main MCU clock references | Rev.A"
- note removed: "Main MCU reset, boot and SWD | Rev.A"
