File: hardware/MIRA_Control/1100_DAC_SERVICE_AND_FORMING.kicad_sch (KiCad schematic)
At the start: 49 parts, among them U1100 AD5676RBRUZ, U1101 OPA4192IPWR, U1102 OPA4192IPWR, U1103 AD5761RBRUZ, U1104 OPA192IDBVR

Commit message: Protect unpowered signal domains and qualify local supplies; retain startup and fault interlocks
MIRA-Startup-Patch: 7ffae17756ebcf923eff1212bb1aade8fbdfae03a9ca8ecebc69d3da3d3b4ba2
Connections:
- net ILIM_FORM_DAC: no longer U1102.10 (+IN)
- net ILIM_RESET_DAC: no longer U1102.5 (+IN)
- net ILIM_SET_DAC: no longer U1102.3 (+IN)
- net MATRIX_BIAS_DAC: no longer U1102.12 (+IN)
- net VREAD_DAC: no longer U1101.3 (+IN)
- net VRESET_DAC: no longer U1101.10 (+IN)
- net VSET_DAC: no longer U1101.5 (+IN)
- net VWL_DAC: no longer U1101.12 (+IN)
- new net ILIM_FORM_DAC_SAFE: U1102.10 (+IN)
- new net ILIM_RESET_DAC_SAFE: U1102.5 (+IN)
- new net ILIM_SET_DAC_SAFE: U1102.3 (+IN)
- new net MATRIX_BIAS_DAC_SAFE: U1102.12 (+IN)
- new net VREAD_DAC_SAFE: U1101.3 (+IN)
- new net VRESET_DAC_SAFE: U1101.10 (+IN)
- new net VSET_DAC_SAFE: U1101.5 (+IN)
- new net VWL_DAC_SAFE: U1101.12 (+IN)
