File: hardware/MIRA_Control/200_MCU_FMC_AND_SDRAM.kicad_sch (KiCad schematic)
At the start: 35 parts, among them U100 STM32H745IIT6, U200 IS42S16320F-7TLI

Commit message: Add high-load schematic candidate with CORE sense and revised N15 supply
Connections:
- net VDD renamed SYS3V3
