File: hardware/MIRA_Control/700_FPGA_USB3_FIFO_INTERFACE.kicad_sch (KiCad schematic)
At the start: 63 parts, among them J700 12401610E4#2A, U500 XC7A200T-2FBG484I, U700 TPD2EUSB30DRTR, U701 TPD2EUSB30DRTR, U702 TPD2EUSB30DRTR, U703 TPD2EUSB30DRTR, U704 TPD2EUSB30DRTR, U705 TPD2EUSB30DRTR, U706 HD3SS3220IRNHR, U707 FT601Q-B-R, U708 74LVC1G17GV, Y700 ABM8-30.000MHZ-B2-T

Commit message: Add high-load schematic candidate with CORE sense and revised N15 supply
Connections:
- net EP renamed GND
- net VCC33 renamed IO3V3
- net VD10 renamed FT1V0

Commit message: Protect unpowered signal domains and qualify local supplies; retain startup and fault interlocks
MIRA-Startup-Patch: 7ffae17756ebcf923eff1212bb1aade8fbdfae03a9ca8ecebc69d3da3d3b4ba2
Connections:
- net GND: no longer U706.29 (ENn_CC)
- net IO3V3: no longer R702.1, U706.8 (VCC33)
- new net USB_CC_DISABLE: U706.29 (ENn_CC)
- new net USB_MUX_3V3: R702.1, U706.8 (VCC33)
Changed lines of the file:
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@@
 	(wire
 		(pts
-			(xy 194.31 189.23) (xy 196.85 189.23)
-		)
-		(stroke
-			(width 0)
-			(type default)
-		)
-	)
-	(wire
-		(pts
 			(xy 121.92 201.93) (xy 121.92 198.12)
 		)
@@
 	(wire
 		(pts
-			(xy 196.85 186.69) (xy 196.85 189.23)
-		)
-		(stroke
-			(width 0)
-			(type default)
-		)
-	)
-	(wire
-		(pts
 			(xy 180.34 250.19) (xy 182.88 250.19)
 		)
@@
 		)
 	)
-	(global_label "IO3V3"
-		(shape bidirectional)
-		(at 137.16 182.88 180)
-		(effects
-			(font
-				(size 0.9 0.9)
-			)
-			(justify right)
-		)
-		(property "Intersheetrefs" "${INTERSHEET_REFS}"
-			(at 137.16 182.88 0)
-			(hide yes)
-			(show_name no)
-			(do_not_autoplace no)
-			(effects
-				(font
-					(size 1 1)
-				)
-			)
-		)
-	)
+	(global_label "USB_MUX_3V3" (shape bidirectional) (at 137.16 182.88 180) (effects (font (size 0.9 0.9)) (justify right)) (property "Intersheetrefs" "${INTERSHEET_REFS}" (at 137.16 182.88 0) (hide yes) (show_name no) (do_not_autoplace no) (effects (font (size 1 1)))))
 	(global_label "USB_RX1_P"
 		(shape bidirectional)
@@
 		)
 	)
-	(global_label "IO3V3"
-		(shape bidirectional)
-		(at 156.21 175.26 180)
-		(effects
-			(font
-				(size 0.9 0.9)
-			)
-			(justify right)
-		)
-		(property "Intersheetrefs" "${INTERSHEET_REFS}"
-			(at 156.21 175.26 0)
-			(hide yes)
-			(show_name no)
-			(do_not_autoplace no)
-			(effects
-				(font
-					(size 1 1)
-				)
-			)
-		)
-	)
+	(global_label "USB_MUX_3V3" (shape bidirectional) (at 156.21 175.26 180) (effects (font (size 0.9 0.9)) (justify right)) (property "Intersheetrefs" "${INTERSHEET_REFS}" (at 156.21 175.26 0) (hide yes) (show_name no) (do_not_autoplace no) (effects (font (size 1 1)))))
 	(global_label "USB_DM"
 		(shape bidirectional)
@@
 		)
 	)
+(global_label "USB_CC_DISABLE" (shape input) (at 194.31 189.23 180) (effects (font (size 0.8 0.8)) (justify right)))
 )
