File: hardware/MIRA_Control/100_MCU_POWER_CLOCKS_AND_DEBUG.kicad_sch (KiCad schematic)
At the start: 46 parts, among them J4801 Cortex SWD 10-pin, J4802 Boot jumper, SW4801 Reset pushbutton, U4101 STM32H745IIT6, Y4801 ASV-25.000MHZ-EJ-T, Y4802 ABS07-32.768KHZ-7-T

Commit message: Replace Control with organized 30-page project
Parts:
- C100: renamed from C4101; Pin assignment U4101 pin 7 VDD -> U100 pin 7 VDD
- C101: renamed from C4102; Pin assignment U4101 pin 13 VDD -> U100 pin 13 VDD
- C102: renamed from C4103; Pin assignment U4101 pin 25 VDD -> U100 pin 25 VDD
- C103: renamed from C4104; Pin assignment U4101 pin 44 VDD -> U100 pin 44 VDD
- C104: renamed from C4105; Pin assignment U4101 pin 48 VDD -> U100 pin 48 VDD
- C105: renamed from C4106; Pin assignment U4101 pin 65 VDD -> U100 pin 65 VDD
- C106: renamed from C4107; Pin assignment U4101 pin 71 VDD -> U100 pin 71 VDD
- C107: renamed from C4108; Pin assignment U4101 pin 84 VDD -> U100 pin 84 VDD
- C108: renamed from C4109; Pin assignment U4101 pin 92 VDD -> U100 pin 92 VDD
- C109: renamed from C4110; Pin assignment U4101 pin 99 VDD -> U100 pin 99 VDD
- C110: renamed from C4111; Pin assignment U4101 pin 105 VDD -> U100 pin 105 VDD
- C111: renamed from C4112; Pin assignment U4101 pin 113 VDD -> U100 pin 113 VDD
- C112: renamed from C4113; Pin assignment U4101 pin 126 VDD -> U100 pin 126 VDD
- C113: renamed from C4114; Pin assignment U4101 pin 136 VDD -> U100 pin 136 VDD
- C114: renamed from C4115; Pin assignment U4101 pin 152 VDD -> U100 pin 152 VDD
- C115: renamed from C4116; Pin assignment U4101 pin 160 VDD -> U100 pin 160 VDD
- C116: renamed from C4117; Pin assignment U4101 pin 176 VDD -> U100 pin 176 VDD
- C117: renamed from C4118; Pin assignment U4101 VDD Bulk reservoir -> U100 VDD Bulk reservoir
- C118: renamed from C4119; Pin assignment U4101 pins 82,135,175 VDDLDO bulk -> U100 pins 82,135,175 VDDLDO bulk
- C119: renamed from C4120; Pin assignment U4101 pin 80 VCAP -> U100 pin 80 VCAP
- C120: renamed from C4121; Pin assignment U4101 pins 133,172 VCAP group -> U100 pins 133,172 VCAP group
- C121: renamed from C4122; Pin assignment U4101 pin 39 VREF+ -> U100 pin 39 VREF+
- C122: renamed from C4123; Pin assignment U4101 pin 39 VREF+ -> U100 pin 39 VREF+
- C123: renamed from C4124; Pin assignment U4101 pin 40 VDDA -> U100 pin 40 VDDA
- C124: renamed from C4125; Pin assignment U4101 pin 40 VDDA -> U100 pin 40 VDDA
- C125: renamed from C4126; Pin assignment U4101 pins 82,135,175 VDDLDO bypass -> U100 pins 82,135,175 VDDLDO bypass
- C126: renamed from C4127; Pin assignment U4101 pin 8 VBAT -> U100 pin 8 VBAT
- C127: renamed from C4128; Pin assignment U4101 pins 120,121 USB supply -> U100 pins 120,121 USB supply
- C128: renamed from C4129; Pin assignment U4101 pin 121 VDD33_USB -> U100 pin 121 VDD33_USB
- C129: renamed from C4801; Pin assignment Y4801 pin 4 VDD -> Y100 pin 4 VDD
- C130: renamed from C4802; Pin assignment U4101 pin 10 LSE_IN / Y4802 pin 1 -> U100 pin 10 LSE_IN / Y101 pin 1
- C131: renamed from C4803; Pin assignment U4101 pin 10 LSE_IN / Y4802 pin 1 -> U100 pin 10 LSE_IN / Y101 pin 1
- C132: renamed from C4804; Pin assignment U4101 pin 33 -> U100 pin 33
- R101: renamed from R4801; Pin assignment U4101 pin 31 / HSE -> U100 pin 31 / HSE
- R102: renamed from R4802; Pin assignment U4101 pin 167 -> U100 pin 167
- R103: renamed from R4803; Pin assignment U4101 pin 132 -> U100 pin 132
- R104: renamed from R4804; Pin assignment U4101 pin 138 -> U100 pin 138
- R105: renamed from R4805; Pin assignment U4101 pin 138 -> U100 pin 138
- R106: renamed from R4806; Pin assignment U4101 pin 33 -> U100 pin 33
- renumbered J4801 to J100, J4802 to J101, R4101 to R100, SW4801 to SW100, U4101 to U100, Y4801 to Y100, Y4802 to Y101
Connections:
- net FPGA_DONE_MCU: now reaches U100.122 (PC6)
- net FPGA_INIT_N_MCU: now reaches U100.123 (PC7)
- no-connect marks 53 -> 51
Other:
- note added: "Clock sources"
- note added: "Filtered supply: source declaration for ERC"
- note added: "Internal core regulator"
- note added: "Local supply bypass"
- note added: "MCU GPIO and FPGA configuration status"
- note added: "MCU GPIO and FPGA configuration status | Rev.A"
- note added: "Processor and supply domains"
- note added: "R106 and C132 bias and filter HOST_RESET_N; SW100 pulls it low. R102 holds BOOT0 low, while J101 permits a high strap. J100 exposes SWD, SWO, reset and the supply reference. R103 and R104 are 33 ohm series resistors in SWD. PC6 (pin 122) receives FPGA_DONE_MCU and PC7 (pin 123) receives FPGA_INIT_N_MCU through the SYS3V3-powered U901 return buffer."
- note added: "Reset, boot and access"
- note added: "STM32 supply, clocks, reset and debug"
- note added: "The 100 nF capacitors provide local bypass paths for the individual supply pins. The 4.7 uF capacitors support the shared rail. The analog, backup and USB supply groups have their own capacitors; their short return paths must be preserved during PCB placement."
- note added: "The three VCAP pins share MCU_VCAP, with C119 and C120 providing two 2.2 uF capacitors to ground. This net is the internal regulator reservoir, not an external supply output. VDDSMPS, VFBSMPS and VSSSMPS are grounded; VLXSMPS is left open in the drawn LDO supply configuration."
- note added: "U100 is the STM32H745 host processor. SYS3V3 supplies VDD, VDDLDO, VBAT and the shown USB supply pins. R100 is a 0 ohm link feeding MCU_VDDA for VDDA and VREF+. The separate MCU units on the other sheets belong to this same physical package."
- note added: "Y100 provides a 25 MHz external clock through the 33 ohm R101 to MCU_HSE_CLK. Y101 is the 32.768 kHz LSE crystal, with 12 pF load capacitors C130 and C131. These two clock networks have different purposes and must be configured accordingly in firmware."
- note removed: "4100_MCU_POWER_CORE"
- note removed: "Control logic"
- note removed: "Do not load MCU_VCAP or connect it to SYS3V3. Check VCAP, NRST and SWD first. USB regulator is disabled; USB pins use SYS3V3."
- note removed: "Inputs and outputs"
- note removed: "LDO-only: VDDSMPS, VFBSMPS and VSSSMPS are GND; VLXSMPS is open. All three VDDLDO pins are connected."
- note removed: "Main MCU reserved GPIO"
- note removed: "Main MCU reserved GPIO | Rev.A"
- note removed: "Main MCU supply and core regulator"
- note removed: "Protection and fault response"
- note removed: "Purpose and role"
- note removed: "SHEET GUIDE / 4100_MCU_POWER_CORE"
- note removed: "Timing and settings"
- note removed: "U4101 runs experiment control and neuron models. The independent AON STM32G0 remains the power manager."
- note removed: "VCAP 80/133/172 share two 2.2u capacitors. Select PWR_LDO_SUPPLY before voltage scaling/PLLs. 480MHz requires VOS0."
- note removed: "VDD, VDDLDO and VBAT use SYS3V3. R4101 feeds VDDA/VREF+. Repeated supply pins are stacked; every physical pin is retained."
- company: (none) -> MIRA
- title: (none) -> STM32 supply, clocks, reset and debug

Commit message: Add high-load schematic candidate with CORE sense and revised N15 supply
Connections:
- net VDD renamed SYS3V3

Commit message: Review MIRA.06 components, connectors and assembly
Parts:
- J100: footprint MIRA_RevA:PinHeader_2x05_P1.27mm_Vertical -> MIRA_RevA:Samtec_FTSH-105-01-L-DV-K_2x05_P1.27mm_SMD
Changed lines of the file:
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@@
 			)
 		)
-		(property "Footprint" "MIRA_RevA:PinHeader_2x05_P1.27mm_Vertical"
+		(property "Footprint" "MIRA_RevA:Samtec_FTSH-105-01-L-DV-K_2x05_P1.27mm_SMD"
 			(at 254 142.24 0)
 			(hide yes)
@@
 			)
 		)
-		(property "Description" "Cortex 10-pin SWD header; VTREF sense only, keyed pin7 unused"
+		(property "Description" "FTSH-105-01-L-DV-K SMT SWD header; pin 7 present and NC; -K keys FFSD housing, does not omit pin 7. Verify debug cable."
 			(at 254 142.24 0)
 			(hide yes)
