File: hardware/MIRA_Control/1800_MATRIX_CROSSBAR_SOCKET_AND_BIAS.kicad_sch (KiCad schematic)
At the start: 5 parts, among them J1800 ICS-CQFP64-1830-1830-100-1, J1801 Bias jumper, J1802 Bias jumper

Commit message: Review MIRA.06 components, connectors and assembly
Parts:
- J1801, J1802: MPN Generic1x3header -> TSW-103-07-G-S; Manufacturer Generic -> Samtec
Changed lines of the file:
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@@
 			)
 		)
-		(property "Datasheet" ""
+		(property "Datasheet" "https://www.samtec.com/products/tsw-103-07-g-s"
 			(at 171.45 96.52 0)
 			(hide yes)
@@
 			)
 		)
-		(property "Description" "Bias jumper"
+		(property "Description" "3-pin 2.54 mm through-hole bias selection header; manual/selective solder after SMT; fit selected 2.54 mm shunt per assembly plan"
 			(at 171.45 96.52 0)
 			(hide yes)
@@
 			)
 		)
-		(property "MPN" "Generic1x3header"
+		(property "MPN" "TSW-103-07-G-S"
 			(at 171.45 96.52 0)
 			(hide yes)
@@
 			)
 		)
-		(property "Manufacturer" "Generic"
+		(property "Manufacturer" "Samtec"
 			(at 171.45 96.52 0)
 			(hide yes)
@@
 			)
 		)
-		(property "Datasheet" ""
-			(at 171.45 57.15 0)
-			(hide yes)
-			(show_name no)
-			(do_not_autoplace no)
-			(effects
-				(font
-					(size 1 1)
-				)
-			)
-		)
-		(property "Description" "Bias jumper"
-			(at 171.45 57.15 0)
-			(hide yes)
-			(show_name no)
-			(do_not_autoplace no)
-			(effects
-				(font
-					(size 1 1)
-				)
-			)
-		)
-		(property "MPN" "Generic1x3header"
-			(at 171.45 57.15 0)
-			(hide yes)
-			(show_name no)
-			(do_not_autoplace no)
-			(effects
-				(font
-					(size 1 1)
-				)
-			)
-		)
-		(property "Manufacturer" "Generic"
-			(at 171.45 57.15 0)
-			(hide yes)
+		(property "Datasheet" "https://www.samtec.com/products/tsw-103-07-g-s"
+			(at 171.45 57.15 0)
+			(hide yes)
+			(show_name no)
+			(do_not_autoplace no)
+			(effects
+				(font
+					(size 1 1)
+				)
+			)
+		)
+		(property "Description" "3-pin 2.54 mm through-hole bias selection header; manual/selective solder after SMT; fit selected 2.54 mm shunt per assembly plan"
+			(at 171.45 57.15 0)
+			(hide yes)
+			(show_name no)
+			(do_not_autoplace no)
+			(effects
+				(font
+					(size 1 1)
+				)
+			)
+		)
+		(property "MPN" "TSW-103-07-G-S"
+			(at 171.45 57.15 0)
+			(hide yes)
+			(show_name no)
+			(do_not_autoplace no)
+			(effects
+				(font
+					(size 1 1)
+				)
+			)
+		)
+		(property "Manufacturer" "Samtec"
+			(at 171.45 57.15 0)
+			(hide yes)
