File: hardware/MIRA_Control/2200_PROTECTION_MATRIX_TRIP_AND_FAULT_INTERFACE.kicad_sch (KiCad schematic)
At the start: 24 parts, among them Q2200 2N7002, Q2201 2N7002, Q2202 BC857B, Q2203 BSS138N, U2200 TLV3201, U2201 SN74LVC1G08, U2202 SN74LVC1G74, U2203 SN74LVC1G32

Commit message: Protect unpowered signal domains and qualify local supplies; retain startup and fault interlocks
MIRA-Startup-Patch: 7ffae17756ebcf923eff1212bb1aade8fbdfae03a9ca8ecebc69d3da3d3b4ba2
Parts:
- R2200: value 49.9k -> 45.3k; MPN TNPW040249K9BEED -> ERJ-2RKF4532X
- R2202: value 37.4k -> 34k; MPN TNPW040237K4BEED -> ERJ-2RKF3402X
Connections:
- net MAT_CMP_N: no longer U2200.4 (IN-)
- net MAT_CMP_P: no longer U2200.3 (IN+)
- new net MAT_CMP_N_SAFE: U2200.4 (IN-)
- new net MAT_CMP_P_SAFE: U2200.3 (IN+)
Changed lines of the file:
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@@
 	(wire
 		(pts
-			(xy 62.23 68.58) (xy 62.23 66.04)
-		)
-		(stroke
-			(width 0)
-			(type default)
-		)
-	)
-	(wire
-		(pts
 			(xy 200.66 127) (xy 200.66 120.65)
 		)
@@
 	(wire
 		(pts
-			(xy 62.23 63.5) (xy 64.77 63.5)
-		)
-		(stroke
-			(width 0)
-			(type default)
-		)
-	)
-	(wire
-		(pts
 			(xy 180.34 124.46) (xy 181.61 124.46)
 		)
@@
 	(wire
 		(pts
-			(xy 62.23 60.96) (xy 62.23 63.5)
-		)
-		(stroke
-			(width 0)
-			(type default)
-		)
-	)
-	(wire
-		(pts
-			(xy 62.23 66.04) (xy 64.77 66.04)
-		)
-		(stroke
-			(width 0)
-			(type default)
-		)
-	)
-	(wire
-		(pts
 			(xy 90.17 62.23) (xy 93.98 62.23)
 		)
@@
 		)
 	)
-	(symbol
-		(lib_id "MIRA_RevA:Resistor")
-		(at 39.37 60.96 90)
-		(unit 1)
-		(body_style 1)
-		(exclude_from_sim no)
-		(in_bom yes)
-		(on_board yes)
-		(in_pos_files yes)
-		(dnp no)
-		(property "Reference" "R2200"
-			(at 39.37 58.46 90)
-			(show_name no)
-			(do_not_autoplace no)
-			(effects
-				(font
-					(size 0.85 0.85)
-				)
-			)
-		)
-		(property "Value" "49.9k"
-			(at 39.37 63.46 90)
-			(show_name no)
-			(do_not_autoplace no)
-			(effects
-				(font
-					(size 0.85 0.85)
-				)
-			)
-		)
-		(property "Footprint" "MIRA_RevA:R_0402_1005Metric"
-			(at 39.37 60.96 0)
-			(hide yes)
-			(show_name no)
-			(do_not_autoplace no)
-			(effects
-				(font
-					(size 1 1)
-				)
-			)
-		)
-		(property "Datasheet" "https://www.vishay.com/docs/28758/tnpw_e3.pdf"
-			(at 39.37 60.96 0)
-			(hide yes)
-			(show_name no)
-			(do_not_autoplace no)
-			(effects
-				(font
-					(size 1 1)
-				)
-			)
-		)
-		(property "Description" "49.9k ohm, 0.1%, 25 ppm/K, precision fault-threshold resistor"
-			(at 39.37 60.96 0)
-			(hide yes)
-			(show_name no)
-			(do_not_autoplace no)
-			(effects
-				(font
-					(size 1 1)
-				)
-			)
-		)
-		(property "MPN" "TNPW040249K9BEED"
-			(at 39.37 60.96 0)
-			(hide yes)
-			(show_name no)
-			(do_not_autoplace no)
-			(effects
-				(font
-					(size 1 1)
-				)
-			)
-		)
-		(property "Manufacturer" "Vishay"
-			(at 39.37 60.96 0)
-			(hide yes)
-			(show_name no)
-			(do_not_autoplace no)
-			(effects
-				(font
-					(size 1 1)
-				)
-			)
-		)
-		(pin "1"
-		)
-		(pin "2"
-		)
-		(instances
-			(project "MIRA_Control"
-				(path "/ad010b50-c509-466c-b833-d1667dfb0702/75a2aa70-81cd-4543-a50c-e295d4f5a68c/c17b5599-39dd-494c-ad64-99a5847f5793"
-					(reference "R2200")
-					(unit 1)
-				)
-			)
-		)
-	)
+	(symbol (lib_id "MIRA_RevA:Resistor") (at 39.37 60.96 90) (unit 1) (body_style 1) (exclude_from_sim no) (in_bom yes) (on_board yes) (in_pos_files yes) (dnp no) (property "Reference" "R2200" (at 39.37 58.46 90) (show_name no) (do_not_autoplace no) (effects (font (size 0.85 0.85)))) (property "Value" "45.3k" (at 39.37 63.46 90) (show_name no) (do_not_autoplace no) (effects (font (size 0.85 0.85)))) (property "Footprint" "MIRA_RevA:R_0402_1005Metric" (at 39.37 60.96 0) (hide yes) (show_name no) (do_not_autoplace no) (effects (font (size 1 1)))) (property "Datasheet" "https://www.vishay.com/docs/28758/tnpw_e3.pdf" (at 39.37 60.96 0) (hide yes) (show_name no) (do_not_autoplace no) (effects (font (size 1 1)))) (property "Description" "49.9k ohm, 0.1%, 25 ppm/K, precision fault-threshold resistor" (at 39.37 60.96 0) (hide yes) (show_name no) (do_not_autoplace no) (effects (font (size 1 1)))) (property "MPN" "ERJ-2RKF4532X" (at 39.37 60.96 0) (hide yes) (show_name no) (do_not_autoplace no) (effects (font (size 1 1)))) (property "Manufacturer" "Vishay" (at 39.37 60.96 0) (hide yes) (show_name no) (do_not_autoplace no) (effects (font (size 1 1)))) (pin "1") (pin "2") (instances (project "MIRA_Control" (path "/ad010b50-c509-466c-b833-d1667dfb0702/75a2aa70-81cd-4543-a50c-e295d4f5a68c/c17b5599-39dd-494c-ad64-99a5847f5793" (reference "R2200") (unit 1)))))
 	(symbol
 		(lib_id "MIRA_RevA:SN74LVC1G08_MIRA_MAT")
@@
 		)
 	)
-	(symbol
-		(lib_id "MIRA_RevA:Resistor")
-		(at 39.37 68.58 90)
-		(unit 1)
-		(body_style 1)
-		(exclude_from_sim no)
-		(in_bom yes)
-		(on_board yes)
-		(in_pos_files yes)
-		(dnp no)
-		(property "Reference" "R2202"
-			(at 39.37 66.08 90)
-			(show_name no)
-			(do_not_autoplace no)
-			(effects
-				(font
-					(size 0.85 0.85)
-				)
-			)
-		)
-		(property "Value" "37.4k"
-			(at 39.37 71.08 90)
-			(show_name no)
-			(do_not_autoplace no)
-			(effects
-				(font
-					(size 0.85 0.85)
-				)
-			)
-		)
-		(property "Footprint" "MIRA_RevA:R_0402_1005Metric"
-			(at 39.37 68.58 0)
-			(hide yes)
-			(show_name no)
-			(do_not_autoplace no)
-			(effects
-				(font
-					(size 1 1)
-				)
-			)
-		)
-		(property "Datasheet" "https://www.vishay.com/docs/28758/tnpw_e3.pdf"
-			(at 39.37 68.58 0)
-			(hide yes)
-			(show_name no)
-			(do_not_autoplace no)
-			(effects
-				(font
-					(size 1 1)
-				)
-			)
-		)
-		(property "Description" "37.4k ohm, 0.1%, 25 ppm/K, precision fault-threshold resistor"
-			(at 39.37 68.58 0)
-			(hide yes)
-			(show_name no)
-			(do_not_autoplace no)
-			(effects
-				(font
-					(size 1 1)
-				)
-			)
-		)
-		(property "MPN" "TNPW040237K4BEED"
-			(at 39.37 68.58 0)
-			(hide yes)
-			(show_name no)
-			(do_not_autoplace no)
-			(effects
-				(font
-					(size 1 1)
-				)
-			)
-		)
-		(property "Manufacturer" "Vishay"
-			(at 39.37 68.58 0)
-			(hide yes)
-			(show_name no)
-			(do_not_autoplace no)
-			(effects
-				(font
-					(size 1 1)
-				)
-			)
-		)
-		(pin "1"
-		)
-		(pin "2"
-		)
-		(instances
-			(project "MIRA_Control"
-				(path "/ad010b50-c509-466c-b833-d1667dfb0702/75a2aa70-81cd-4543-a50c-e295d4f5a68c/c17b5599-39dd-494c-ad64-99a5847f5793"
-					(reference "R2202")
-					(unit 1)
-				)
-			)
-		)
-	)
+	(symbol (lib_id "MIRA_RevA:Resistor") (at 39.37 68.58 90) (unit 1) (body_style 1) (exclude_from_sim no) (in_bom yes) (on_board yes) (in_pos_files yes) (dnp no) (property "Reference" "R2202" (at 39.37 66.08 90) (show_name no) (do_not_autoplace no) (effects (font (size 0.85 0.85)))) (property "Value" "34k" (at 39.37 71.08 90) (show_name no) (do_not_autoplace no) (effects (font (size 0.85 0.85)))) (property "Footprint" "MIRA_RevA:R_0402_1005Metric" (at 39.37 68.58 0) (hide yes) (show_name no) (do_not_autoplace no) (effects (font (size 1 1)))) (property "Datasheet" "https://www.vishay.com/docs/28758/tnpw_e3.pdf" (at 39.37 68.58 0) (hide yes) (show_name no) (do_not_autoplace no) (effects (font (size 1 1)))) (property "Description" "37.4k ohm, 0.1%, 25 ppm/K, precision fault-threshold resistor" (at 39.37 68.58 0) (hide yes) (show_name no) (do_not_autoplace no) (effects (font (size 1 1)))) (property "MPN" "ERJ-2RKF3402X" (at 39.37 68.58 0) (hide yes) (show_name no) (do_not_autoplace no) (effects (font (size 1 1)))) (property "Manufacturer" "Vishay" (at 39.37 68.58 0) (hide yes) (show_name no) (do_not_autoplace no) (effects (font (size 1 1)))) (pin "1") (pin "2") (instances (project "MIRA_Control" (path "/ad010b50-c509-466c-b833-d1667dfb0702/75a2aa70-81cd-4543-a50c-e295d4f5a68c/c17b5599-39dd-494c-ad64-99a5847f5793" (reference "R2202") (unit 1)))))
 	(symbol
 		(lib_id "MIRA_RevA:2N7002_MIRA_MAT")
@@
 		)
 	)
+(global_label "MAT_CMP_P_SAFE" (shape input) (at 64.77 63.5 180) (effects (font (size 0.8 0.8)) (justify right)))
+(global_label "MAT_CMP_N_SAFE" (shape input) (at 64.77 66.04 180) (effects (font (size 0.8 0.8)) (justify right)))
 )

Commit message: MIRA.05: analog requirements and schematic fixes
Parts:
- R2200, R2202: Manufacturer Vishay -> Panasonic
Other:
- note added: "Backup trip nominal: 1.25623 x ILIM + 0.09397 V WRITE qualified only; READ / VMM have no such trip."
- note added: "R2200/R2201 = 45.3k/10k; R2202/R2203 = 34k/10k. Include both 100k guard bleeds on sheet 3000 and R2211=1.5M from IO3V3. Nominal backup trip: VSENSE > 1.25623*VILIM + 0.09397 V at IO3V3=3.3 V. This is coarse shutdown, not precision CC. Comparator offset, leakage and resistor tolerances add error."
- note removed: "Backup trip only: 1.2571 x ILIM + 0.10343 V Current regulation and pulse energy are evaluated on sheet 2100."
- note removed: "R2200/R2201 = 49.9k/10k divide normalized source-current sense by 5.99. R2202/R2203 = 37.4k/10k and R2211 = 1.5M from IO3V3 set the backup threshold. Nominal trip: VSENSE > 1.2571*VILIM + 0.10343 V. The CV/CC loop is the precision current regulator; this comparator is independent coarse shutdown."
Changed lines of the file:
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@@
 		)
 	)
-	(text "R2200/R2201 = 49.9k/10k divide normalized source-current\nsense by 5.99. R2202/R2203 = 37.4k/10k and R2211 = 1.5M\nfrom IO3V3 set the backup threshold. Nominal trip: VSENSE\n> 1.2571*VILIM + 0.10343 V. The CV/CC loop is the\nprecision current regulator; this comparator is\nindependent coarse shutdown."
-		(exclude_from_sim no)
-		(at 22.86 174.34 0)
-		(effects
-			(font
-				(size 1.1 1.1)
-				(color 0 70 160 1)
-			)
-			(justify left top)
-		)
-	)
+	(text "R2200/R2201 = 45.3k/10k; R2202/R2203 = 34k/10k.\nInclude both 100k guard bleeds on sheet 3000 and\nR2211=1.5M from IO3V3. Nominal backup trip:\nVSENSE > 1.25623*VILIM + 0.09397 V at IO3V3=3.3 V.\nThis is coarse shutdown, not precision CC. Comparator\noffset, leakage and resistor tolerances add error." (exclude_from_sim no) (at 22.86 174.34 0) (effects (font (size 1.1 1.1) (color 0 70 160 1)) (justify left top)))
 	(text "MATRIX_INHIBIT_N to Power / connector sheet 400"
 		(exclude_from_sim no)
@@
 		)
 	)
-	(text "Backup trip only: 1.2571 x ILIM + 0.10343 V\nCurrent regulation and pulse energy are evaluated on sheet 2100."
-		(exclude_from_sim no)
-		(at 22.86 83.82 0)
-		(effects
-			(font
-				(size 1.05 1.05)
-				(color 0 70 160 1)
-			)
-			(justify left top)
-		)
-	)
+	(text "Backup trip nominal: 1.25623 x ILIM + 0.09397 V\nWRITE qualified only; READ / VMM have no such trip." (exclude_from_sim no) (at 22.86 83.82 0) (effects (font (size 1.05 1.05) (color 0 70 160 1)) (justify left top)))
 	(text "Clocked trip memory / asynchronous clear"
 		(exclude_from_sim no)
@@
 		)
 	)
-	(symbol (lib_id "MIRA_RevA:Resistor") (at 39.37 60.96 90) (unit 1) (body_style 1) (exclude_from_sim no) (in_bom yes) (on_board yes) (in_pos_files yes) (dnp no) (property "Reference" "R2200" (at 39.37 58.46 90) (show_name no) (do_not_autoplace no) (effects (font (size 0.85 0.85)))) (property "Value" "45.3k" (at 39.37 63.46 90) (show_name no) (do_not_autoplace no) (effects (font (size 0.85 0.85)))) (property "Footprint" "MIRA_RevA:R_0402_1005Metric" (at 39.37 60.96 0) (hide yes) (show_name no) (do_not_autoplace no) (effects (font (size 1 1)))) (property "Datasheet" "https://www.vishay.com/docs/28758/tnpw_e3.pdf" (at 39.37 60.96 0) (hide yes) (show_name no) (do_not_autoplace no) (effects (font (size 1 1)))) (property "Description" "49.9k ohm, 0.1%, 25 ppm/K, precision fault-threshold resistor" (at 39.37 60.96 0) (hide yes) (show_name no) (do_not_autoplace no) (effects (font (size 1 1)))) (property "MPN" "ERJ-2RKF4532X" (at 39.37 60.96 0) (hide yes) (show_name no) (do_not_autoplace no) (effects (font (size 1 1)))) (property "Manufacturer" "Vishay" (at 39.37 60.96 0) (hide yes) (show_name no) (do_not_autoplace no) (effects (font (size 1 1)))) (pin "1") (pin "2") (instances (project "MIRA_Control" (path "/ad010b50-c509-466c-b833-d1667dfb0702/75a2aa70-81cd-4543-a50c-e295d4f5a68c/c17b5599-39dd-494c-ad64-99a5847f5793" (reference "R2200") (unit 1)))))
+	(symbol (lib_id "MIRA_RevA:Resistor") (at 39.37 60.96 90) (unit 1) (body_style 1) (exclude_from_sim no) (in_bom yes) (on_board yes) (in_pos_files yes) (dnp no) (property "Reference" "R2200" (at 39.37 58.46 90) (show_name no) (do_not_autoplace no) (effects (font (size 0.85 0.85)))) (property "Value" "45.3k" (at 39.37 63.46 90) (show_name no) (do_not_autoplace no) (effects (font (size 0.85 0.85)))) (property "Footprint" "MIRA_RevA:R_0402_1005Metric" (at 39.37 60.96 0) (hide yes) (show_name no) (do_not_autoplace no) (effects (font (size 1 1)))) (property "Datasheet" "https://industrial.panasonic.com/ww/products/pt/general-purpose-chip-resistors/models/ERJ2RKF4532X" (at 39.37 60.96 0) (hide yes) (show_name no) (do_not_autoplace no) (effects (font (size 1 1)))) (property "Description" "45.3k ohm, 1%, 0402; Panasonic ERJ-2RKF; calibrate actual divider ratio" (at 39.37 60.96 0) (hide yes) (show_name no) (do_not_autoplace no) (effects (font (size 1 1)))) (property "MPN" "ERJ-2RKF4532X" (at 39.37 60.96 0) (hide yes) (show_name no) (do_not_autoplace no) (effects (font (size 1 1)))) (property "Manufacturer" "Panasonic" (at 39.37 60.96 0) (hide yes) (show_name no) (do_not_autoplace no) (effects (font (size 1 1)))) (pin "1") (pin "2") (instances (project "MIRA_Control" (path "/ad010b50-c509-466c-b833-d1667dfb0702/75a2aa70-81cd-4543-a50c-e295d4f5a68c/c17b5599-39dd-494c-ad64-99a5847f5793" (reference "R2200") (unit 1)))))
 	(symbol
 		(lib_id "MIRA_RevA:SN74LVC1G08_MIRA_MAT")
@@
 		)
 	)
-	(symbol (lib_id "MIRA_RevA:Resistor") (at 39.37 68.58 90) (unit 1) (body_style 1) (exclude_from_sim no) (in_bom yes) (on_board yes) (in_pos_files yes) (dnp no) (property "Reference" "R2202" (at 39.37 66.08 90) (show_name no) (do_not_autoplace no) (effects (font (size 0.85 0.85)))) (property "Value" "34k" (at 39.37 71.08 90) (show_name no) (do_not_autoplace no) (effects (font (size 0.85 0.85)))) (property "Footprint" "MIRA_RevA:R_0402_1005Metric" (at 39.37 68.58 0) (hide yes) (show_name no) (do_not_autoplace no) (effects (font (size 1 1)))) (property "Datasheet" "https://www.vishay.com/docs/28758/tnpw_e3.pdf" (at 39.37 68.58 0) (hide yes) (show_name no) (do_not_autoplace no) (effects (font (size 1 1)))) (property "Description" "37.4k ohm, 0.1%, 25 ppm/K, precision fault-threshold resistor" (at 39.37 68.58 0) (hide yes) (show_name no) (do_not_autoplace no) (effects (font (size 1 1)))) (property "MPN" "ERJ-2RKF3402X" (at 39.37 68.58 0) (hide yes) (show_name no) (do_not_autoplace no) (effects (font (size 1 1)))) (property "Manufacturer" "Vishay" (at 39.37 68.58 0) (hide yes) (show_name no) (do_not_autoplace no) (effects (font (size 1 1)))) (pin "1") (pin "2") (instances (project "MIRA_Control" (path "/ad010b50-c509-466c-b833-d1667dfb0702/75a2aa70-81cd-4543-a50c-e295d4f5a68c/c17b5599-39dd-494c-ad64-99a5847f5793" (reference "R2202") (unit 1)))))
+	(symbol (lib_id "MIRA_RevA:Resistor") (at 39.37 68.58 90) (unit 1) (body_style 1) (exclude_from_sim no) (in_bom yes) (on_board yes) (in_pos_files yes) (dnp no) (property "Reference" "R2202" (at 39.37 66.08 90) (show_name no) (do_not_autoplace no) (effects (font (size 0.85 0.85)))) (property "Value" "34k" (at 39.37 71.08 90) (show_name no) (do_not_autoplace no) (effects (font (size 0.85 0.85)))) (property "Footprint" "MIRA_RevA:R_0402_1005Metric" (at 39.37 68.58 0) (hide yes) (show_name no) (do_not_autoplace no) (effects (font (size 1 1)))) (property "Datasheet" "https://industrial.panasonic.com/ww/products/pt/general-purpose-chip-resistors/models/ERJ2RKF3402X" (at 39.37 68.58 0) (hide yes) (show_name no) (do_not_autoplace no) (effects (font (size 1 1)))) (property "Description" "34k ohm, 1%, 0402; Panasonic ERJ-2RKF; calibrate actual divider ratio" (at 39.37 68.58 0) (hide yes) (show_name no) (do_not_autoplace no) (effects (font (size 1 1)))) (property "MPN" "ERJ-2RKF3402X" (at 39.37 68.58 0) (hide yes) (show_name no) (do_not_autoplace no) (effects (font (size 1 1)))) (property "Manufacturer" "Panasonic" (at 39.37 68.58 0) (hide yes) (show_name no) (do_not_autoplace no) (effects (font (size 1 1)))) (pin "1") (pin "2") (instances (project "MIRA_Control" (path "/ad010b50-c509-466c-b833-d1667dfb0702/75a2aa70-81cd-4543-a50c-e295d4f5a68c/c17b5599-39dd-494c-ad64-99a5847f5793" (reference "R2202") (unit 1)))))
 	(symbol
 		(lib_id "MIRA_RevA:2N7002_MIRA_MAT")

Commit message: Review MIRA.06 components, connectors and assembly
Parts:
- Q2203: MPN BSS138N -> BSS138NH6327XTSA2
Changed lines of the file:
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@@
 			)
 		)
-		(property "Datasheet" "https://www.infineon.com/dgdl/Infineon-BSS138N-DataSheet-v02_00-EN.pdf"
+		(property "Datasheet" "https://www.infineon.com/part/BSS138N"
 			(at 208.28 127 0)
 			(hide yes)
@@
 			)
 		)
-		(property "MPN" "BSS138N"
+		(property "MPN" "BSS138NH6327XTSA2"
 			(at 208.28 127 0)
 			(hide yes)
