File: hardware/MIRA_Control/archive/UNUSED_SCHEMATIC_SOURCES/3300 - Matrix adapter and bias configuration.kicad_sch (KiCad schematic)
At the start: 5 parts, among them J8001 Matrix adapter 2x32, J8002 Bias jumper, J8003 Bias jumper

Commit message: Replace Control with organized 30-page project
Parts:
- J8001: value Matrix adapter 2x32 -> ICS-CQFP64-1830-1830-100-1; footprint MIRA_RevA:PinHeader_2x32_P2.54mm_Vertical -> MIRA_RevA:ICS-CQFP64-1830-1830-100-1; symbol MIRA_RevA:Matrix_adapter_2x32_MIRA_MAT -> MIRA_RevA:ICS_CQFP64_1830_1830_100_1_MIRA; MPN Generic2x32header -> ICS-CQFP64-1830-1830-100-1; Manufacturer Generic -> IC SOCKET
Connections:
- net MAT_ADAPTER_CASE: now also J8001.40 (CASE_COM); no longer J8001.48
- net MAT_ADAPTER_VSUB: now also J8001.48 (GND_REF); no longer J8001.40
Other:
- note added: "BL routing: 2200-2500 WL drivers: 2700 | NL selection / clamps: 2800 MATRIX_BIAS_SRC: 1800 J8001A and J8001B are one 64-contact socket. BL0-BL15 use contacts 64-49 in reverse order. Pin 40: CASE_COM. Pin 48: GND in the user reference; its existing configurable net is MAT_ADAPTER_VSUB. Default both bias selectors to GND. Unused NC contacts are not permanent GND."
- note added: "Crossbar socket and bias configuration"
- note added: "Pin 48 / Reference GND or bias"
- note removed: "BL routing: 2200-2500 WL drivers: 2700 | NL selection / clamps: 2800 MATRIX_BIAS_SRC: 1800 J8001A and J8001B are units of the same connector. BL0-BL15 use contacts 64-49 in reverse contact order. VSUB: contact 40 | CASE: contact 48 Unused NC contacts are not permanent GND."
- note removed: "Matrix adapter and bias configuration"
- note removed: "Substrate / Select GND or bias"
Changed lines of the file:
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@@
 	(generator_version "10.0")
 	(paper "A3")
-	(text "Matrix adapter and bias configuration"
+	(text "Crossbar socket and bias configuration"
 		(exclude_from_sim no)
 		(at 22.86 20.955 0)
@@
 		)
 	)
-	(text "BL routing: 2200-2500\nWL drivers: 2700   |   NL selection / clamps: 2800\nMATRIX_BIAS_SRC: 1800\n\nJ8001A and J8001B are units of the same connector.\nBL0-BL15 use contacts 64-49 in reverse contact order.\nVSUB: contact 40   |   CASE: contact 48\nUnused NC contacts are not permanent GND."
+	(text "BL routing: 2200-2500\nWL drivers: 2700   |   NL selection / clamps: 2800\nMATRIX_BIAS_SRC: 1800\n\nJ8001A and J8001B are one 64-contact socket.\nBL0-BL15 use contacts 64-49 in reverse order.\nPin 40: CASE_COM. Pin 48: GND in the user reference;\nits existing configurable net is MAT_ADAPTER_VSUB.\nDefault both bias selectors to GND.\nUnused NC contacts are not permanent GND."
 		(exclude_from_sim no)
 		(at 142.24 125.73 0)
@@
 		)
 	)
-	(text "Substrate / Select GND or bias"
+	(text "Pin 48 / Reference GND or bias"
 		(exclude_from_sim no)
 		(at 142.24 37.465 0)
@@
 		)
 	)
+	(global_label "MAT_ADAPTER_CASE"
+		(shape bidirectional)
+		(at 100.33 66.04 180)
+		(effects
+			(font
+				(size 0.9 0.9)
+			)
+			(justify right)
+		)
+		(property "Intersheetrefs" "${INTERSHEET_REFS}"
+			(at 100.33 66.04 0)
+			(hide yes)
+			(show_name no)
+			(do_not_autoplace no)
+			(effects
+				(font
+					(size 1 1)
+				)
+			)
+		)
+	)
 	(global_label "MAT_ADAPTER_VSUB"
-		(shape bidirectional)
-		(at 100.33 66.04 180)
-		(effects
-			(font
-				(size 0.9 0.9)
-			)
-			(justify right)
-		)
-		(property "Intersheetrefs" "${INTERSHEET_REFS}"
-			(at 100.33 66.04 0)
-			(hide yes)
-			(show_name no)
-			(do_not_autoplace no)
-			(effects
-				(font
-					(size 1 1)
-				)
-			)
-		)
-	)
-	(global_label "MAT_ADAPTER_CASE"
 		(shape bidirectional)
 		(at 100.33 86.36 180)
@@
 	)
 	(symbol
-		(lib_id "MIRA_RevA:Matrix_adapter_2x32_MIRA_MAT")
+		(lib_id "MIRA_RevA:ICS_CQFP64_1830_1830_100_1_MIRA")
 		(at 46.99 87.63 0)
 		(unit 1)
@@
 			)
 		)
-		(property "Value" "Matrix adapter 2x32"
+		(property "Value" "ICS-CQFP64-1830-1830-100-1"
 			(at 46.99 132.08 0)
 			(show_name no)
@@
 			)
 		)
-		(property "Footprint" "MIRA_RevA:PinHeader_2x32_P2.54mm_Vertical"
+		(property "Footprint" "MIRA_RevA:ICS-CQFP64-1830-1830-100-1"
 			(at 46.99 87.63 0)
 			(hide yes)
@@
 			)
 		)
-		(property "Datasheet" ""
+		(property "Datasheet" "https://icsocket.ru/ku/cqfp/489"
 			(at 46.99 87.63 0)
 			(hide yes)
@@
 			)
 		)
-		(property "Description" "Standard 2x32 carrier interface; source-map numbering, no invented matrix package"
+		(property "Description" "64-contact IC SOCKET for the crossbar; pin map follows the user reference"
 			(at 46.99 87.63 0)
 			(hide yes)
@@
 			)
 		)
-		(property "MPN" "Generic2x32header"
+		(property "MPN" "ICS-CQFP64-1830-1830-100-1"
 			(at 46.99 87.63 0)
 			(hide yes)
@@
 			)
 		)
-		(property "Manufacturer" "Generic"
+		(property "Manufacturer" "IC SOCKET"
 			(at 46.99 87.63 0)
 			(hide yes)
@@
 	)
 	(symbol
-		(lib_id "MIRA_RevA:Matrix_adapter_2x32_MIRA_MAT")
+		(lib_id "MIRA_RevA:ICS_CQFP64_1830_1830_100_1_MIRA")
 		(at 110.49 87.63 0)
 		(unit 2)
@@
 			)
 		)
-		(property "Value" "Matrix adapter 2x32"
+		(property "Value" "ICS-CQFP64-1830-1830-100-1"
 			(at 110.49 132.08 0)
 			(show_name no)
@@
 			)
 		)
-		(property "Footprint" "MIRA_RevA:PinHeader_2x32_P2.54mm_Vertical"
+		(property "Footprint" "MIRA_RevA:ICS-CQFP64-1830-1830-100-1"
 			(at 110.49 87.63 0)
 			(hide yes)
@@
 			)
 		)
-		(property "Datasheet" ""
+		(property "Datasheet" "https://icsocket.ru/ku/cqfp/489"
 			(at 110.49 87.63 0)
 			(hide yes)
@@
 			)
 		)
-		(property "Description" "Standard 2x32 carrier interface; source-map numbering, no invented matrix package"
+		(property "Description" "64-contact IC SOCKET for the crossbar; pin map follows the user reference"
 			(at 110.49 87.63 0)
 			(hide yes)
@@
 			)
 		)
-		(property "MPN" "Generic2x32header"
+		(property "MPN" "ICS-CQFP64-1830-1830-100-1"
 			(at 110.49 87.63 0)
 			(hide yes)
@@
 			)
 		)
-		(property "Manufacturer" "Generic"
+		(property "Manufacturer" "IC SOCKET"
 			(at 110.49 87.63 0)
 			(hide yes)
