File: hardware/MIRA_Power/1000_AFE_POSITIVE_15V.kicad_sch (KiCad schematic)
At the start: 16 parts, among them Q1001 BSS138N, U1001 LMR51610XDBVR

Commit message: Protect unpowered signal domains and qualify local supplies; retain startup and fault interlocks
MIRA-Startup-Patch: 7ffae17756ebcf923eff1212bb1aade8fbdfae03a9ca8ecebc69d3da3d3b4ba2
Connections:
- net EN_P15: no longer U1001.4 (EN)
- new net EN_P15_VIN: U1001.4 (EN)
Changed lines of the file:
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@@
-	(wire
-		(pts
-			(xy 66.04 85.09) (xy 66.04 96.52)
-		)
-		(stroke
-			(width 0)
-			(type default)
-		)
-	)
 	(wire
 		(pts
@@
 		(pts
 			(xy 83.82 83.82) (xy 83.82 82.55)
-		)
-		(stroke
-			(width 0)
-			(type default)
-		)
-	)
-	(wire
-		(pts
-			(xy 66.04 96.52) (xy 63.5 96.52)
 		)
 		(stroke
@@
 		)
 	)
+(global_label "EN_P15_VIN" (shape input) (at 63.5 96.52 180) (effects (font (size 0.8 0.8)) (justify right)))
 )
