File: hardware/MIRA_Power/1400_FPGA_AUX_2V5.kicad_sch (KiCad schematic)
At the start: 13 parts, among them Q1401 BSS138N, U1401 TPS62130ARGTR

Commit message: Protect unpowered signal domains and qualify local supplies; retain startup and fault interlocks
MIRA-Startup-Patch: 7ffae17756ebcf923eff1212bb1aade8fbdfae03a9ca8ecebc69d3da3d3b4ba2
Connections:
- net EN_AUX25: no longer U1401.13 (EN)
- new net EN_AUX25_VIN: U1401.13 (EN)
Changed lines of the file:
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@@
 		)
 	)
-	(global_label "EN_AUX25"
-		(shape input)
-		(at 52.07 115.57 180)
-		(effects
-			(font
-				(size 1 1)
-			)
-			(justify right)
-		)
-		(property "Intersheetrefs" "${INTERSHEET_REFS}"
-			(at 52.07 115.57 0)
-			(hide yes)
-			(show_name no)
-			(do_not_autoplace no)
-			(effects
-				(font
-					(size 1 1)
-				)
-			)
-		)
-	)
+	(global_label "EN_AUX25_VIN" (shape input) (at 52.07 115.57 180) (effects (font (size 1 1)) (justify right)) (property "Intersheetrefs" "${INTERSHEET_REFS}" (at 52.07 115.57 0) (hide yes) (show_name no) (do_not_autoplace no) (effects (font (size 1 1)))))
 	(global_label "AUX2V5"
 		(shape input)
