File: hardware/MIRA_Power/1600_DDR_1V35.kicad_sch (KiCad schematic)
At the start: 13 parts, among them Q1601 BSS138N, U1601 TPS62130ARGTR

Commit message: Protect unpowered signal domains and qualify local supplies; retain startup and fault interlocks
MIRA-Startup-Patch: 7ffae17756ebcf923eff1212bb1aade8fbdfae03a9ca8ecebc69d3da3d3b4ba2
Connections:
- net EN_DDR: no longer U1601.13 (EN)
- new net EN_DDR_VIN: U1601.13 (EN)
Changed lines of the file:
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@@
 		)
 	)
-	(global_label "EN_DDR"
-		(shape input)
-		(at 52.07 115.57 180)
-		(effects
-			(font
-				(size 1 1)
-			)
-			(justify right)
-		)
-		(property "Intersheetrefs" "${INTERSHEET_REFS}"
-			(at 52.07 115.57 0)
-			(hide yes)
-			(show_name no)
-			(do_not_autoplace no)
-			(effects
-				(font
-					(size 1 1)
-				)
-			)
-		)
-	)
+	(global_label "EN_DDR_VIN" (shape input) (at 52.07 115.57 180) (effects (font (size 1 1)) (justify right)) (property "Intersheetrefs" "${INTERSHEET_REFS}" (at 52.07 115.57 0) (hide yes) (show_name no) (do_not_autoplace no) (effects (font (size 1 1)))))
 	(global_label "DDR_RAW"
 		(shape input)
