File: hardware/MIRA_Power/2400_PM_CONTROLLER.kicad_sch (KiCad schematic)
At the start: 6 parts, among them U2401 STM32G0B1RBT6

Commit message: Add high-load schematic candidate with CORE sense and revised N15 supply
Parts:
- U2401: gpio_map {'1': {'gpio': 'PC11', 'net': 'PWR_KILL_GPIO'}, '2': {'gpio': 'PC12', 'net': 'MATRIX_KILL_GPIO'}, '3': {'gpio': 'PC13', 'net': 'ALL_RAILS_PG'}, '4': {'gpio': 'PC14', 'net': None}, '5': {'gpio': 'PC15', 'net': None}, '6': {'gpio': 'VBAT', 'net': 'AON'}, '7': {'gpio': 'VREF+', 'net': 'AON'}, '8': {'gpio': 'VDD/VDDA', 'net': 'AON'}, '9': {'gpio': 'VSS/VSSA', 'net': 'GND'}, '10': {'gpio': 'PF0', 'net': 'EN_REQ_USB'}, '11': {'gpio': 'PF1', 'net': None}, '12': {'gpio': 'PF2/NRST', 'net': 'PM_RESET_N'}, '13': {'gpio': 'PC0', 'net': 'PWR_ARM_PULSE'}, '14': {'gpio': 'PC1', 'net': 'MATRIX_ARM_PULSE'}, '15': {'gpio': 'PC2', 'net': 'PM_WDI'}, '16': {'gpio': 'PC3', 'net': 'PM_WDO_N'}, '17': {'gpio': 'PA0', 'net': 'ADC_I'}, '18': {'gpio': 'PA1', 'net': 'ADC_V'}, '19': {'gpio': 'PA2', 'net': 'ADC_VTT'}, '20': {'gpio': 'PA3', 'net': 'PROG_V_P15'}, '21': {'gpio': 'PA4', 'net': 'EN_REQ_SYS'}, '22': {'gpio': 'PA5', 'net': 'EN_REQ_FPGA'}, '23': {'gpio': 'PA6', 'net': 'EN_REQ_ANA'}, '24': {'gpio': 'PA7', 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 -> {'1': {'gpio': 'PC11', 'net': 'PWR_KILL_GPIO'}, '2': {'gpio': 'PC12', 'net': 'MATRIX_KILL_GPIO'}, '3': {'gpio': 'PC13', 'net': 'ALL_RAILS_PG'}, '4': {'gpio': 'PC14', 'net': None}, '5': {'gpio': 'PC15', 'net': None}, '6': {'gpio': 'VBAT', 'net': 'AON'}, '7': {'gpio': 'VREF+', 'net': 'AON'}, '8': {'gpio': 'VDD/VDDA', 'net': 'AON'}, '9': {'gpio': 'VSS/VSSA', 'net': 'GND'}, '10': {'gpio': 'PF0', 'net': 'EN_REQ_USB'}, '11': {'gpio': 'PF1', 'net': 'HOST_ALIVE_PM'}, '12': {'gpio': 'PF2/NRST', 'net': 'PM_RESET_N'}, '13': {'gpio': 'PC0', 'net': 'PWR_ARM_PULSE'}, '14': {'gpio': 'PC1', 'net': 'MATRIX_ARM_PULSE'}, '15': {'gpio': 'PC2', 'net': 'PM_WDI'}, '16': {'gpio': 'PC3', 'net': 'PM_WDO_N'}, '17': {'gpio': 'PA0', 'net': 'ADC_I'}, '18': {'gpio': 'PA1', 'net': 'ADC_V'}, '19': {'gpio': 'PA2', 'net': 'ADC_VTT'}, '20': {'gpio': 'PA3', 'net': 'PROG_V_P15'}, '21': {'gpio': 'PA4', 'net': 'EN_REQ_SYS'}, '22': {'gpio': 'PA5', 'net': 'EN_REQ_FPGA'}, '23': {'gpio': 'PA6', 'net': 'EN_REQ_ANA'}, '24': {'gpi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
Connections:
- net HOST_ALIVE_PM: now reaches U2401.11 (PF1)
- no-connect marks 3 -> 2
Changed lines of the file:
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@@
 	)
 	(no_connect
-		(at 90.17 74.93)
-	)
-	(no_connect
 		(at 90.17 59.69)
 	)
@@
 			)
 		)
-		(property "gpio_map" "{'1': {'gpio': 'PC11', 'net': 'PWR_KILL_GPIO'}, '2': {'gpio': 'PC12', 'net': 'MATRIX_KILL_GPIO'}, '3': {'gpio': 'PC13', 'net': 'ALL_RAILS_PG'}, '4': {'gpio': 'PC14', 'net': None}, '5': {'gpio': 'PC15', 'net': None}, '6': {'gpio': 'VBAT', 'net': 'AON'}, '7': {'gpio': 'VREF+', 'net': 'AON'}, '8': {'gpio': 'VDD/VDDA', 'net': 'AON'}, '9': {'gpio': 'VSS/VSSA', 'net': 'GND'}, '10': {'gpio': 'PF0', 'net': 'EN_REQ_USB'}, '11': {'gpio': 'PF1', 'net': None}, '12': {'gpio': 'PF2/NRST', 'net': 'PM_RESET_N'}, '13': {'gpio': 'PC0', 'net': 'PWR_ARM_PULSE'}, '14': {'gpio': 'PC1', 'net': 'MATRIX_ARM_PULSE'}, '15': {'gpio': 'PC2', 'net': 'PM_WDI'}, '16': {'gpio': 'PC3', 'net': 'PM_WDO_N'}, '17': {'gpio': 'PA0', 'net': 'ADC_I'}, '18': {'gpio': 'PA1', 'net': 'ADC_V'}, '19': {'gpio': 'PA2', 'net': 'ADC_VTT'}, '20': {'gpio': 'PA3', 'net': 'PROG_V_P15'}, '21': {'gpio': 'PA4', 'net': 'EN_REQ_SYS'}, '22': {'gpio': 'PA5', 'net': 'EN_REQ_FPGA'}, '23': {'gpio': 'PA6', 'net': 'EN_REQ_ANA'}, '24': {'gpio': 'PA7', 'net': 'EN_REQ_P15'}, '25': {'gpio': 'PC4', 'net': 'EN_REQ_N15'}, '26': {'gpio': 'PC5', 'net': 'EN_REQ_CORE'}, '27': {'gpio': 'PB0', 'net': 'EN_REQ_AUX18'}, '28': {'gpio': 'PB1', 'net': 'EN_REQ_AUX25'}, '29': {'gpio': 'PB2', 'net': 'EN_REQ_IO33'}, '30': {'gpio': 'PB10', 'net': 'EN_REQ_DDR'}, '31': {'gpio': 'PB11', 'net': 'EN_REQ_PHY'}, '32': {'gpio': 'PB12', 'net': 'EN_REQ_VTT'}, '33': {'gpio': 'PB13', 'net': 'EN_REQ_ANA5'}, '34': {'gpio': 'PB14', 'net': 'EN_REQ_ANA33'}, '35': {'gpio': 'PB15', 'net': 'MUX_A0'}, '36': {'gpio': 'PA8', 'net': 'MUX_A1'}, '37': {'gpio': 'PA9', 'net': 'MUX_A2'}, '38': {'gpio': 'PC6', 'net': 'MUX_A3'}, '39': {'gpio': 'PC7', 'net': 'MUX_DISABLE'}, '40': {'gpio': 'PD8', 'net': 'PM_UART_TX'}, '41': {'gpio': 'PD9', 'net': 'PM_UART_RX'}, '42': {'gpio': 'PA10', 'net': 'PG_INPUT'}, '43': {'gpio': 'PA11', 'net': 'FLT_INPUT_N'}, '44': {'gpio': 'PA12', 'net': 'OC_OK_N'}, '45': {'gpio': 'PA13/SWDIO', 'net': 'PM_SWDIO_MCU'}, '46': {'gpio': 'PA14/BOOT0/SWCLK', 'net': 'PM_SWCLK_MCU'}, '47': {'gpio': 'PA15', 'net': 'GLOBAL_PWR_PERMIT'}, '48': {'gpio': 'PC8', 'net': 'MATRIX_PERMIT'}, '49': {'gpio': 'PC9', 'net': 'HOST_WDO_N'}, '50': {'gpio': 'PD0', 'net': 'PG_USB'}, '51': {'gpio': 'PD1', 'net': 'PG_SYS'}, '52': {'gpio': 'PD2', 'net': 'PG_FPGA'}, '53': {'gpio': 'PD3', 'net': 'PG_ANA'}, '54': {'gpio': 'PD4', 'net': 'PG_P15'}, '55': {'gpio': 'PD5', 'net': 'PG_N15'}, '56': {'gpio': 'PD6', 'net': 'PGR_CORE'}, '57': {'gpio': 'PB3', 'net': 'PGR_AUX18'}, '58': {'gpio': 'PB4', 'net': 'PGR_AUX25'}, '59': {'gpio': 'PB5', 'net': 'PGR_IO33'}, '60': {'gpio': 'PB6', 'net': 'PGR_DDR'}, '61': {'gpio': 'PB7', 'net': 'PGR_PHY'}, '62': {'gpio': 'PB8', 'net': 'PGR_VTT'}, '63': {'gpio': 'PB9', 'net': 'PGR_ANA5'}, '64': {'gpio': 'PC10', 'net': 'PGR_ANA33'}}"
+		(property "gpio_map" "{'1': {'gpio': 'PC11', 'net': 'PWR_KILL_GPIO'}, '2': {'gpio': 'PC12', 'net': 'MATRIX_KILL_GPIO'}, '3': {'gpio': 'PC13', 'net': 'ALL_RAILS_PG'}, '4': {'gpio': 'PC14', 'net': None}, '5': {'gpio': 'PC15', 'net': None}, '6': {'gpio': 'VBAT', 'net': 'AON'}, '7': {'gpio': 'VREF+', 'net': 'AON'}, '8': {'gpio': 'VDD/VDDA', 'net': 'AON'}, '9': {'gpio': 'VSS/VSSA', 'net': 'GND'}, '10': {'gpio': 'PF0', 'net': 'EN_REQ_USB'}, '11': {'gpio': 'PF1', 'net': 'HOST_ALIVE_PM'}, '12': {'gpio': 'PF2/NRST', 'net': 'PM_RESET_N'}, '13': {'gpio': 'PC0', 'net': 'PWR_ARM_PULSE'}, '14': {'gpio': 'PC1', 'net': 'MATRIX_ARM_PULSE'}, '15': {'gpio': 'PC2', 'net': 'PM_WDI'}, '16': {'gpio': 'PC3', 'net': 'PM_WDO_N'}, '17': {'gpio': 'PA0', 'net': 'ADC_I'}, '18': {'gpio': 'PA1', 'net': 'ADC_V'}, '19': {'gpio': 'PA2', 'net': 'ADC_VTT'}, '20': {'gpio': 'PA3', 'net': 'PROG_V_P15'}, '21': {'gpio': 'PA4', 'net': 'EN_REQ_SYS'}, '22': {'gpio': 'PA5', 'net': 'EN_REQ_FPGA'}, '23': {'gpio': 'PA6', 'net': 'EN_REQ_ANA'}, '24': {'gpio': 'PA7', 'net': 'EN_REQ_P15'}, '25': {'gpio': 'PC4', 'net': 'EN_REQ_N15'}, '26': {'gpio': 'PC5', 'net': 'EN_REQ_CORE'}, '27': {'gpio': 'PB0', 'net': 'EN_REQ_AUX18'}, '28': {'gpio': 'PB1', 'net': 'EN_REQ_AUX25'}, '29': {'gpio': 'PB2', 'net': 'EN_REQ_IO33'}, '30': {'gpio': 'PB10', 'net': 'EN_REQ_DDR'}, '31': {'gpio': 'PB11', 'net': 'EN_REQ_PHY'}, '32': {'gpio': 'PB12', 'net': 'EN_REQ_VTT'}, '33': {'gpio': 'PB13', 'net': 'EN_REQ_ANA5'}, '34': {'gpio': 'PB14', 'net': 'EN_REQ_ANA33'}, '35': {'gpio': 'PB15', 'net': 'MUX_A0'}, '36': {'gpio': 'PA8', 'net': 'MUX_A1'}, '37': {'gpio': 'PA9', 'net': 'MUX_A2'}, '38': {'gpio': 'PC6', 'net': 'MUX_A3'}, '39': {'gpio': 'PC7', 'net': 'MUX_DISABLE'}, '40': {'gpio': 'PD8', 'net': 'PM_UART_TX'}, '41': {'gpio': 'PD9', 'net': 'PM_UART_RX'}, '42': {'gpio': 'PA10', 'net': 'PG_INPUT'}, '43': {'gpio': 'PA11', 'net': 'FLT_INPUT_N'}, '44': {'gpio': 'PA12', 'net': 'OC_OK_N'}, '45': {'gpio': 'PA13/SWDIO', 'net': 'PM_SWDIO_MCU'}, '46': {'gpio': 'PA14/BOOT0/SWCLK', 'net': 'PM_SWCLK_MCU'}, '47': {'gpio': 'PA15', 'net': 'GLOBAL_PWR_PERMIT'}, '48': {'gpio': 'PC8', 'net': 'MATRIX_PERMIT'}, '49': {'gpio': 'PC9', 'net': 'HOST_WDO_N'}, '50': {'gpio': 'PD0', 'net': 'PG_USB'}, '51': {'gpio': 'PD1', 'net': 'PG_SYS'}, '52': {'gpio': 'PD2', 'net': 'PG_FPGA'}, '53': {'gpio': 'PD3', 'net': 'PG_ANA'}, '54': {'gpio': 'PD4', 'net': 'PG_P15'}, '55': {'gpio': 'PD5', 'net': 'PG_N15'}, '56': {'gpio': 'PD6', 'net': 'PGR_CORE'}, '57': {'gpio': 'PB3', 'net': 'PGR_AUX18'}, '58': {'gpio': 'PB4', 'net': 'PGR_AUX25'}, '59': {'gpio': 'PB5', 'net': 'PGR_IO33'}, '60': {'gpio': 'PB6', 'net': 'PGR_DDR'}, '61': {'gpio': 'PB7', 'net': 'PGR_PHY'}, '62': {'gpio': 'PB8', 'net': 'PGR_VTT'}, '63': {'gpio': 'PB9', 'net': 'PGR_ANA5'}, '64': {'gpio': 'PC10', 'net': 'PGR_ANA33'}}"
 			(at 107.95 88.9 0)
 			(hide yes)
@@
 		)
 	)
+(wire (pts (xy 90.17 74.93) (xy 82.55 74.93)) (stroke (width 0) (type default)))
+(global_label "HOST_ALIVE_PM" (shape input) (at 82.55 74.93 180) (effects (font (size 1.016 1.016)) (justify right)))
 )

Commit message: Protect unpowered signal domains and qualify local supplies; retain startup and fault interlocks
MIRA-Startup-Patch: 7ffae17756ebcf923eff1212bb1aade8fbdfae03a9ca8ecebc69d3da3d3b4ba2
Connections:
- net GLOBAL_CLEAR_N: now reaches U2401.4 (PC14)
- net LINK_READY_H: now reaches U2401.5 (PC15)
- net ADC_VTT renamed ADC_VTT_SAFE
- no-connect marks 2 -> 0
Other:
- note added: "PC14: GLOBAL_CLEAR_N; PC15: LINK_READY_H. Inputs, no pull; LSE OFF. Wait for CLEAR before PWR_ARM; LINK_READY before MATRIX_ARM. Read HOST_ALIVE_PM as a heartbeat; verify both permit outputs."
- note added: "Wait for PC14 CLEAR before PWR_ARM; PC15 LINK_READY before MATRIX_ARM. Service PM_WDI throughout startup and shutdown. Use internal clocking; PF0, PC14 and PC15 are GPIO, not HSE/LSE. See docs/pcb-preparation/sequencing/README.md for rail order."
- note removed: "Read GLOBAL_PWR_PERMIT and MATRIX_PERMIT as inputs. Initialize EN_REQ_* safely before applying either arm pulse."
- note removed: "The startup order and rail settling delays are set in firmware. Service PM_WDI before the external watchdog can time out. Use internal clocking: PF0 is assigned to EN_REQ_USB. Keep NRST and SWD active; keep the VREFBUF output disabled."
Changed lines of the file:
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@@
 		)
 	)
-	(text "Read GLOBAL_PWR_PERMIT and MATRIX_PERMIT as inputs.\nInitialize EN_REQ_* safely before applying either arm pulse."
+	(text "PC14: GLOBAL_CLEAR_N; PC15: LINK_READY_H. Inputs, no pull; LSE OFF.\nWait for CLEAR before PWR_ARM; LINK_READY before MATRIX_ARM.\nRead HOST_ALIVE_PM as a heartbeat; verify both permit outputs."
 		(exclude_from_sim no)
 		(at 20.32 140.335 0)
@@
 		)
 	)
-	(text "The startup order and rail settling delays are set in firmware.\nService PM_WDI before the external watchdog can time out.\nUse internal clocking: PF0 is assigned to EN_REQ_USB.\nKeep NRST and SWD active; keep the VREFBUF output disabled."
+	(text "Wait for PC14 CLEAR before PWR_ARM; PC15 LINK_READY before MATRIX_ARM.\nService PM_WDI throughout startup and shutdown.\nUse internal clocking; PF0, PC14 and PC15 are GPIO, not HSE/LSE.\nSee docs/pcb-preparation/sequencing/README.md for rail order."
 		(exclude_from_sim no)
 		(at 156.21 114.02 0)
@@
 		(color 0 0 0 0)
 	)
-	(no_connect
-		(at 90.17 59.69)
-	)
-	(no_connect
-		(at 90.17 57.15)
-	)
 	(wire
 		(pts
@@
 		)
 	)
-	(global_label "ADC_VTT"
-		(shape input)
-		(at 81.28 95.25 180)
-		(effects
-			(font
-				(size 1 1)
-			)
-			(justify right)
-		)
-		(property "Intersheetrefs" "${INTERSHEET_REFS}"
-			(at 81.28 95.25 0)
-			(hide yes)
-			(show_name no)
-			(do_not_autoplace no)
-			(effects
-				(font
-					(size 1 1)
-				)
-			)
-		)
-	)
+	(global_label "ADC_VTT_SAFE" (shape input) (at 81.28 95.25 180) (effects (font (size 1 1)) (justify right)) (property "Intersheetrefs" "${INTERSHEET_REFS}" (at 81.28 95.25 0) (hide yes) (show_name no) (do_not_autoplace no) (effects (font (size 1 1)))))
 	(global_label "ADC_V"
 		(shape input)
@@
 		)
 	)
-(wire (pts (xy 90.17 74.93) (xy 82.55 74.93)) (stroke (width 0) (type default)))
-(global_label "HOST_ALIVE_PM" (shape input) (at 82.55 74.93 180) (effects (font (size 1.016 1.016)) (justify right)))
+	(wire (pts (xy 90.17 74.93) (xy 82.55 74.93)) (stroke (width 0) (type default)))
+	(global_label "HOST_ALIVE_PM" (shape input) (at 82.55 74.93 180) (effects (font (size 1.016 1.016)) (justify right)))
+	(wire
+		(pts
+			(xy 80.01 57.15)
+			(xy 90.17 57.15)
+		)
+		(stroke
+			(width 0)
+			(type default)
+		)
+	)
+	(global_label "GLOBAL_CLEAR_N"
+		(shape input)
+		(at 80.01 57.15 0)
+		(effects
+			(font
+				(size 1 1)
+			)
+			(justify right)
+		)
+		(property "Intersheetrefs" "${INTERSHEET_REFS}"
+			(at 81.28 54.61 0)
+			(hide yes)
+			(show_name no)
+			(do_not_autoplace no)
+			(effects
+				(font
+					(size 1 1)
+				)
+			)
+		)
+	)
+	(wire
+		(pts
+			(xy 80.01 59.69)
+			(xy 90.17 59.69)
+		)
+		(stroke
+			(width 0)
+			(type default)
+		)
+	)
+	(global_label "LINK_READY_H"
+		(shape input)
+		(at 80.01 59.69 0)
+		(effects
+			(font
+				(size 1 1)
+			)
+			(justify right)
+		)
+		(property "Intersheetrefs" "${INTERSHEET_REFS}"
+			(at 81.28 54.61 0)
+			(hide yes)
+			(show_name no)
+			(do_not_autoplace no)
+			(effects
+				(font
+					(size 1 1)
+				)
+			)
+		)
+	)
 )
