File: hardware/MIRA_Power/2500_PM_WATCHDOGS.kicad_sch (KiCad schematic)
At the start: 17 parts, among them J2501 PM MANUAL RESET CONTACT, J2502 HOST MANUAL RESET CONTACT, U2501 TPS3851H33EDRBR, U2502 TPS3851H33EDRBR

Commit message: Add high-load schematic candidate with CORE sense and revised N15 supply
Connections:
- net AON: no longer R2509.2
- net SYS3V3: now also R2509.2
Changed lines of the file:
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@@
 	)
 	(junction
-		(at 119.38 120.65)
-		(diameter 0)
-		(color 0 0 0 0)
-	)
-	(junction
 		(at 119.38 33.02)
 		(diameter 0)
@@
 	(wire
 		(pts
-			(xy 119.38 120.65) (xy 132.08 120.65)
-		)
-		(stroke
-			(width 0)
-			(type default)
-		)
-	)
-	(wire
-		(pts
 			(xy 101.6 139.7) (xy 104.14 139.7)
 		)
@@
 	(wire
 		(pts
-			(xy 132.08 121.92) (xy 132.08 120.65)
-		)
-		(stroke
-			(width 0)
-			(type default)
-		)
-	)
-	(wire
-		(pts
 			(xy 55.88 34.29) (xy 55.88 35.56)
 		)
@@
 		)
 	)
+(wire (pts (xy 132.08 121.92) (xy 132.08 116.84)) (stroke (width 0) (type default)))
+(global_label "SYS3V3" (shape input) (at 132.08 116.84 0) (effects (font (size 1.016 1.016)) (justify left)))
 )

Commit message: Protect unpowered signal domains and qualify local supplies; retain startup and fault interlocks
MIRA-Startup-Patch: 7ffae17756ebcf923eff1212bb1aade8fbdfae03a9ca8ecebc69d3da3d3b4ba2
Other:
- note added: "AON reset or PM watchdog fault pulls the PM controller reset low. Host reset coupling is on sheet 5400."
- note added: "D2501 combines AON_RESET_N and PM_WDO_N into PM_RESET_N. Either LOW resets U2401 through the common-anode diode. Host WDO now also pulls HOST_RESET_N LOW through U5405 on sheet 5400; both host faults clear matrix permission."
- note added: "J2502 requests a host manual reset. R2509 pulls HOST_RESET_N to SYS3V3, not AON."
- note added: "Supply undervoltage or manual reset asserts RESET. PM expiry resets PM; host expiry also resets host via U5405. HOST_RESET_N pullups stay on SYS3V3; WDO pullups use AON. Sheet 5400 adds application-heartbeat timeout and first-edge latch."
- note removed: "AON reset or PM watchdog fault pulls the controller reset low. Host fault signals stay separate."
- note removed: "D2501 combines AON_RESET_N and PM_WDO_N into PM_RESET_N. Either low signal resets U2401 through the common-anode diode. Host watchdog and reset signals remain separate on this sheet; the hardware interlocks use them to qualify matrix operation."
- note removed: "J2502 requests a host manual reset. AON pullups retain the control-domain logic level."
- note removed: "Supply undervoltage or a shorted manual contact asserts RESET. Watchdog expiry asserts WDO; PM expiry also resets the MCU. AON pullups make status readable in the control domain. Host rail readiness must also inhibit operation while SYS3V3 is off."
Changed lines of the file:
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@@
 		)
 	)
-	(text "AON reset or PM watchdog fault\npulls the controller reset low.\nHost fault signals stay separate."
+	(text "AON reset or PM watchdog fault\npulls the PM controller reset low.\nHost reset coupling is on sheet 5400."
 		(exclude_from_sim no)
 		(at 20.32 86.36 0)
@@
 		)
 	)
-	(text "D2501 combines AON_RESET_N and PM_WDO_N into PM_RESET_N.\nEither low signal resets U2401 through the common-anode diode.\nHost watchdog and reset signals remain separate on this sheet;\nthe hardware interlocks use them to qualify matrix operation."
+	(text "D2501 combines AON_RESET_N and PM_WDO_N into PM_RESET_N.\nEither LOW resets U2401 through the common-anode diode.\nHost WDO now also pulls HOST_RESET_N LOW through U5405\non sheet 5400; both host faults clear matrix permission."
 		(exclude_from_sim no)
 		(at 156.21 91.16 0)
@@
 		)
 	)
-	(text "Supply undervoltage or a shorted manual contact asserts RESET.\nWatchdog expiry asserts WDO; PM expiry also resets the MCU.\nAON pullups make status readable in the control domain.\nHost rail readiness must also inhibit operation while SYS3V3 is off."
+	(text "Supply undervoltage or manual reset asserts RESET.\nPM expiry resets PM; host expiry also resets host via U5405.\nHOST_RESET_N pullups stay on SYS3V3; WDO pullups use AON.\nSheet 5400 adds application-heartbeat timeout and first-edge latch."
 		(exclude_from_sim no)
 		(at 156.21 136.88 0)
@@
 		)
 	)
-	(text "J2502 requests a host manual reset.\nAON pullups retain the control-domain logic level."
+	(text "J2502 requests a host manual reset.\nR2509 pulls HOST_RESET_N to SYS3V3, not AON."
 		(exclude_from_sim no)
 		(at 20.32 112.395 0)
@@
 		)
 	)
-(wire (pts (xy 132.08 121.92) (xy 132.08 116.84)) (stroke (width 0) (type default)))
-(global_label "SYS3V3" (shape input) (at 132.08 116.84 0) (effects (font (size 1.016 1.016)) (justify left)))
+	(wire (pts (xy 132.08 121.92) (xy 132.08 116.84)) (stroke (width 0) (type default)))
+	(global_label "SYS3V3" (shape input) (at 132.08 116.84 0) (effects (font (size 1.016 1.016)) (justify left)))
 )
