File: hardware/MIRA_Power/2600_PM_PERMIT_INTERLOCKS.kicad_sch (KiCad schematic)
At the start: 18 parts, among them J2601 GLOBAL STOP - CLOSE TO TRIP, J2602 MATRIX STOP - CLOSE TO TRIP, J2603 MATRIX HARDWARE INTERLOCK - A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, Q2601 BSS138N, Q2602 BSS138N, U2601 SN74HCS21PWR, U2602 SN74HCS21PWR, U2603 SN74HC74PWR

Commit message: Add high-load schematic candidate with CORE sense and revised N15 supply
Connections:
- net MATRIX_INHIBIT_N: now reaches J2602.2 (Pin_2), Q2602.3 (D), R2605.1, U2602.12 (2C)
Changed lines of the file:
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@@
 		)
 	)
+(global_label "MATRIX_INHIBIT_N" (shape input) (at 57.15 115.57 0) (effects (font (size 1.016 1.016)) (justify left)))
 )

Commit message: Protect unpowered signal domains and qualify local supplies; retain startup and fault interlocks
MIRA-Startup-Patch: 7ffae17756ebcf923eff1212bb1aade8fbdfae03a9ca8ecebc69d3da3d3b4ba2
Connections:
- net AON: no longer U2602.13 (2D)
- net GLOBAL_CLEAR_N: no longer U2601.8 (2Y)
- net MATRIX_PERMIT: no longer U2603.9 (2Q)
- net HOST_RESET_N renamed HOST_RESET_AON_N
- new net GLOBAL_CLEAR_RAW_N: U2601.8 (2Y)
- new net LINK_READY_H: U2602.13 (2D)
- new net MATRIX_PERMIT_RAW: U2603.9 (2Q)
Other:
- note added: "A global fault clears both permissions; a matrix fault clears only matrix permission. Fault recovery alone does not re-arm either latch. Sheets 5200/5300 block startup outputs and qualify GLOBAL_CLEAR_N. AON_RESET_N remains in the clear chain. The stop connectors trip when closed; an open cable is not detected as a stop."
- note added: "Global inputs cover input power, AON reset, PM watchdog/reset, overcurrent and global stop. Matrix inputs add rail/command readiness, host watchdog/reset, LINK_READY_H and matrix stop. J2603 exports MATRIX_PERMIT and raw MATRIX_KILL_H. Application heartbeat qualification is on sheet 5400."
- note removed: "A global fault clears both permissions; a matrix fault clears only matrix permission. Fault recovery alone does not re-arm either latch. AON_RESET_N must clear U2603 during startup. The stop connectors trip when closed; an open cable is not detected as a stop."
- note removed: "Global inputs cover input power, AON reset, PM watchdog/reset, overcurrent and the global stop. Matrix inputs add rail/command readiness, host watchdog/reset and the matrix stop. J2603 exports MATRIX_PERMIT, its inverse MATRIX_KILL_H, AON and GND."
Changed lines of the file:
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@@
 		)
 	)
-	(text "A global fault clears both permissions; a matrix fault clears only\nmatrix permission. Fault recovery alone does not re-arm either latch.\nAON_RESET_N must clear U2603 during startup. The stop connectors\ntrip when closed; an open cable is not detected as a stop."
+	(text "A global fault clears both permissions; a matrix fault clears only\nmatrix permission. Fault recovery alone does not re-arm either latch.\nSheets 5200/5300 block startup outputs and qualify GLOBAL_CLEAR_N.\nAON_RESET_N remains in the clear chain. The stop connectors trip\nwhen closed; an open cable is not detected as a stop."
 		(exclude_from_sim no)
 		(at 156.21 136.88 0)
@@
 		)
 	)
-	(text "Global inputs cover input power, AON reset, PM watchdog/reset,\novercurrent and the global stop. Matrix inputs add rail/command\nreadiness, host watchdog/reset and the matrix stop. J2603 exports\nMATRIX_PERMIT, its inverse MATRIX_KILL_H, AON and GND."
+	(text "Global inputs cover input power, AON reset, PM watchdog/reset,\novercurrent and global stop. Matrix inputs add rail/command\nreadiness, host watchdog/reset, LINK_READY_H and matrix stop.\nJ2603 exports MATRIX_PERMIT and raw MATRIX_KILL_H.\nApplication heartbeat qualification is on sheet 5400."
 		(exclude_from_sim no)
 		(at 156.21 68.3 0)
@@
 		)
 	)
-	(label "GLOBAL_CLEAR_N"
+	(global_label "GLOBAL_CLEAR_RAW_N"
+		(shape bidirectional)
 		(at 125.73 55.88 0)
 		(effects
@@
 		)
 	)
-	(label "GLOBAL_CLEAR_N"
+	(global_label "GLOBAL_CLEAR_N"
+		(shape bidirectional)
 		(at 77.47 144.78 180)
 		(effects
@@
 		)
 	)
-	(global_label "AON"
+	(global_label "LINK_READY_H"
 		(shape input)
 		(at 87.63 118.11 180)
@@
 		)
 	)
-	(global_label "MATRIX_PERMIT"
+	(global_label "MATRIX_PERMIT_RAW"
 		(shape input)
 		(at 124.46 176.53 0)
@@
 		)
 	)
-	(global_label "HOST_RESET_N"
+	(global_label "HOST_RESET_AON_N"
 		(shape input)
 		(at 87.63 113.03 180)
@@
 		)
 	)
-(global_label "MATRIX_INHIBIT_N" (shape input) (at 57.15 115.57 0) (effects (font (size 1.016 1.016)) (justify left)))
+	(global_label "MATRIX_INHIBIT_N" (shape input) (at 57.15 115.57 0) (effects (font (size 1.016 1.016)) (justify left)))
 )
