File: hardware/MIRA_Power/2700_PM_ENABLE_GATES_PRIMARY.kicad_sch (KiCad schematic)
At the start: 20 parts, among them U2701 SN74HC08PWR, U2702 SN74HC08PWR

Commit message: Protect unpowered signal domains and qualify local supplies; retain startup and fault interlocks
MIRA-Startup-Patch: 7ffae17756ebcf923eff1212bb1aade8fbdfae03a9ca8ecebc69d3da3d3b4ba2
Connections:
- net CMD_ANA renamed CMD_ANA_RAW
- net CMD_AUX18 renamed CMD_AUX18_RAW
- net CMD_CORE renamed CMD_CORE_RAW
- net CMD_FPGA renamed CMD_FPGA_RAW
- net CMD_N15 renamed CMD_N15_RAW
- net CMD_P15 renamed CMD_P15_RAW
- net CMD_SYS renamed CMD_SYS_RAW
- net CMD_USB renamed CMD_USB_RAW
Other:
- note added: "Every channel uses the same rule: CMD_x_RAW = GLOBAL_PWR_PERMIT AND EN_REQ_x. Sheet 5300 passes these commands only after STARTUP_READY_H. The power manager chooses the sequence and explicitly arms permits."
- note added: "Raw CMD = request AND global permit; qualified on sheet 5300"
- note added: "U2701 generates CMD_USB_RAW, CMD_SYS_RAW, CMD_FPGA_RAW and CMD_ANA_RAW. U2702 generates CMD_P15_RAW, CMD_N15_RAW, CMD_CORE_RAW and CMD_AUX18_RAW. Each channel receives GLOBAL_PWR_PERMIT and its corresponding EN_REQ signal from the power manager."
- note removed: "Every CMD = request AND global permit"
- note removed: "Every channel uses the same rule: CMD_x = GLOBAL_PWR_PERMIT AND EN_REQ_x. Both inputs must be HIGH to enable the rail. The power manager chooses the sequence; these gates add the hardware permission."
- note removed: "U2701 generates CMD_USB, CMD_SYS, CMD_FPGA and CMD_ANA. U2702 generates CMD_P15, CMD_N15, CMD_CORE and CMD_AUX18. Each channel receives GLOBAL_PWR_PERMIT and its corresponding EN_REQ signal from the power manager."
Changed lines of the file:
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@@
 		)
 	)
-	(text "Every channel uses the same rule:\nCMD_x = GLOBAL_PWR_PERMIT AND EN_REQ_x.\nBoth inputs must be HIGH to enable the rail. The power manager\nchooses the sequence; these gates add the hardware permission."
+	(text "Every channel uses the same rule:\nCMD_x_RAW = GLOBAL_PWR_PERMIT AND EN_REQ_x.\nSheet 5300 passes these commands only after STARTUP_READY_H.\nThe power manager chooses the sequence and explicitly arms permits."
 		(exclude_from_sim no)
 		(at 156.21 91.16 0)
@@
 		)
 	)
-	(text "U2701 generates CMD_USB, CMD_SYS, CMD_FPGA and CMD_ANA.\nU2702 generates CMD_P15, CMD_N15, CMD_CORE and CMD_AUX18.\nEach channel receives GLOBAL_PWR_PERMIT and its corresponding\nEN_REQ signal from the power manager."
+	(text "U2701 generates CMD_USB_RAW, CMD_SYS_RAW, CMD_FPGA_RAW and CMD_ANA_RAW.\nU2702 generates CMD_P15_RAW, CMD_N15_RAW, CMD_CORE_RAW and CMD_AUX18_RAW.\nEach channel receives GLOBAL_PWR_PERMIT and its corresponding\nEN_REQ signal from the power manager."
 		(exclude_from_sim no)
 		(at 156.21 68.3 0)
@@
 		)
 	)
-	(text "Every CMD = request AND global permit"
+	(text "Raw CMD = request AND global permit; qualified on sheet 5300"
 		(exclude_from_sim no)
 		(at 18 193 0)
@@
 		)
 	)
-	(global_label "CMD_N15"
+	(global_label "CMD_N15_RAW"
 		(shape input)
 		(at 128.27 139.7 0)
@@
 		)
 	)
-	(global_label "CMD_FPGA"
+	(global_label "CMD_FPGA_RAW"
 		(shape input)
 		(at 128.27 72.39 0)
@@
 		)
 	)
-	(global_label "CMD_USB"
+	(global_label "CMD_USB_RAW"
 		(shape input)
 		(at 128.27 31.75 0)
@@
 		)
 	)
-	(global_label "CMD_SYS"
+	(global_label "CMD_SYS_RAW"
 		(shape input)
 		(at 128.27 52.07 0)
@@
 		)
 	)
-	(global_label "CMD_ANA"
+	(global_label "CMD_ANA_RAW"
 		(shape input)
 		(at 128.27 92.71 0)
@@
 		)
 	)
-	(global_label "CMD_P15"
+	(global_label "CMD_P15_RAW"
 		(shape input)
 		(at 128.27 119.38 0)
@@
 		)
 	)
-	(global_label "CMD_AUX18"
+	(global_label "CMD_AUX18_RAW"
 		(shape input)
 		(at 128.27 180.34 0)
@@
 		)
 	)
-	(global_label "CMD_CORE"
+	(global_label "CMD_CORE_RAW"
 		(shape input)
 		(at 128.27 160.02 0)
