File: hardware/MIRA_Power/2800_PM_ENABLE_GATES_AUXILIARY.kicad_sch (KiCad schematic)
At the start: 18 parts, among them U2801 SN74HC08PWR, U2802 SN74HC08PWR

Commit message: Protect unpowered signal domains and qualify local supplies; retain startup and fault interlocks
MIRA-Startup-Patch: 7ffae17756ebcf923eff1212bb1aade8fbdfae03a9ca8ecebc69d3da3d3b4ba2
Connections:
- net CMD_ANA33 renamed CMD_ANA33_RAW
- net CMD_ANA5 renamed CMD_ANA5_RAW
- net CMD_AUX25 renamed CMD_AUX25_RAW
- net CMD_DDR renamed CMD_DDR_RAW
- net CMD_IO33 renamed CMD_IO33_RAW
- net CMD_PHY renamed CMD_PHY_RAW
- net CMD_VTT renamed CMD_VTT_RAW
Other:
- note added: "Each used channel follows the same rule: CMD_x_RAW = GLOBAL_PWR_PERMIT AND EN_REQ_x. Sheet 5300 also requires STARTUP_READY_H before outputs are driven. The unused U2802 inputs are grounded and its output is not connected."
- note added: "Raw CMD = request AND global permit; qualified on sheet 5300"
- note added: "U2801 generates CMD_AUX25_RAW, CMD_IO33_RAW, CMD_DDR_RAW and CMD_PHY_RAW. U2802 generates CMD_VTT_RAW, CMD_ANA5_RAW and CMD_ANA33_RAW. Each used channel receives GLOBAL_PWR_PERMIT and its matching EN_REQ input. The fourth U2802 gate is unused."
- note removed: "Each used channel follows the same rule: CMD_x = GLOBAL_PWR_PERMIT AND EN_REQ_x. The request selects a rail; the permit authorizes its operation. The unused U2802 inputs are grounded and its output is not connected."
- note removed: "Every CMD = request AND global permit"
- note removed: "U2801 generates CMD_AUX25, CMD_IO33, CMD_DDR and CMD_PHY. U2802 generates CMD_VTT, CMD_ANA5 and CMD_ANA33. Each used channel receives GLOBAL_PWR_PERMIT and its matching EN_REQ input. The fourth U2802 gate is unused."
Changed lines of the file:
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@@
 		)
 	)
-	(text "Each used channel follows the same rule:\nCMD_x = GLOBAL_PWR_PERMIT AND EN_REQ_x.\nThe request selects a rail; the permit authorizes its operation.\nThe unused U2802 inputs are grounded and its output is not connected."
+	(text "Each used channel follows the same rule:\nCMD_x_RAW = GLOBAL_PWR_PERMIT AND EN_REQ_x.\nSheet 5300 also requires STARTUP_READY_H before outputs are driven.\nThe unused U2802 inputs are grounded and its output is not connected."
 		(exclude_from_sim no)
 		(at 156.21 91.16 0)
@@
 		)
 	)
-	(text "U2801 generates CMD_AUX25, CMD_IO33, CMD_DDR and CMD_PHY.\nU2802 generates CMD_VTT, CMD_ANA5 and CMD_ANA33.\nEach used channel receives GLOBAL_PWR_PERMIT and its matching\nEN_REQ input. The fourth U2802 gate is unused."
+	(text "U2801 generates CMD_AUX25_RAW, CMD_IO33_RAW, CMD_DDR_RAW and CMD_PHY_RAW.\nU2802 generates CMD_VTT_RAW, CMD_ANA5_RAW and CMD_ANA33_RAW.\nEach used channel receives GLOBAL_PWR_PERMIT and its matching\nEN_REQ input. The fourth U2802 gate is unused."
 		(exclude_from_sim no)
 		(at 156.21 68.3 0)
@@
 		)
 	)
-	(text "Every CMD = request AND global permit"
+	(text "Raw CMD = request AND global permit; qualified on sheet 5300"
 		(exclude_from_sim no)
 		(at 18 193 0)
@@
 		)
 	)
-	(global_label "CMD_DDR"
+	(global_label "CMD_DDR_RAW"
 		(shape input)
 		(at 128.27 72.39 0)
@@
 		)
 	)
-	(global_label "CMD_ANA5"
+	(global_label "CMD_ANA5_RAW"
 		(shape input)
 		(at 128.27 139.7 0)
@@
 		)
 	)
-	(global_label "CMD_ANA33"
+	(global_label "CMD_ANA33_RAW"
 		(shape input)
 		(at 128.27 160.02 0)
@@
 		)
 	)
-	(global_label "CMD_AUX25"
+	(global_label "CMD_AUX25_RAW"
 		(shape input)
 		(at 128.27 31.75 0)
@@
 		)
 	)
-	(global_label "CMD_VTT"
+	(global_label "CMD_VTT_RAW"
 		(shape input)
 		(at 128.27 119.38 0)
@@
 		)
 	)
-	(global_label "CMD_PHY"
+	(global_label "CMD_PHY_RAW"
 		(shape input)
 		(at 128.27 92.71 0)
@@
 		)
 	)
-	(global_label "CMD_IO33"
+	(global_label "CMD_IO33_RAW"
 		(shape input)
 		(at 128.27 52.07 0)
