File: hardware/MIRA_Power/300_INPUT_EFUSE_PROTECTION.kicad_sch (KiCad schematic)
At the start: 21 parts, among them Q301 IRFR3410, Q302 BSS138N, U301 TPS26631PWPR

Commit message: Add high-load schematic candidate with CORE sense and revised N15 supply
Parts:
- R301: value 12k -> 13.7k; MPN RC0402FR-0712KL -> RT0402BRD0713K7L
- R302: value 16k -> 14.3k; MPN RC0402FR-0716KL -> RT0402BRD0714K3L
Other:
- note added: "R301=13.7k / R302=14.3k (0.1%, 25ppm/K) protect the 36 V module. Nominal UVLO turn-on remains 16.63 V; OVP cutoff is now 33.99 V. Nominal recovery from OVP is 31.78 V. Design input: 24 V nominal; 18-30 V continuous candidate range, not the former 18-36 V assumption. R305=5.1k and MODE latch-off are unchanged. Validate surge let-through and all tolerance/temperature corners before hardware release."
- note removed: "R301-R304 set the input operating window: approximately 16.63 V turn-on and 38.80 V overvoltage cutoff. Hysteresis gives approximately 15.55 V undervoltage shutdown and 36.28 V recovery from overvoltage. R305 (5.1 kOhm) sets the nominal current limit to 3.53 A. After power-good asserts, TPS26631 permits approximately 7.06 A for a nominal 25.5 ms pulse. MODE is open, selecting latch-off after a su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"
Changed lines of the file:
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@@
 		)
 	)
-	(text "R301-R304 set the input operating window: approximately 16.63 V turn-on\nand 38.80 V overvoltage cutoff. Hysteresis gives approximately 15.55 V\nundervoltage shutdown and 36.28 V recovery from overvoltage.\nR305 (5.1 kOhm) sets the nominal current limit to 3.53 A. After power-good\nasserts, TPS26631 permits approximately 7.06 A for a nominal 25.5 ms pulse.\nMODE is open, selecting latch-off after a sustained overload."
+	(text "R301=13.7k / R302=14.3k (0.1%, 25ppm/K) protect the 36 V module.\nNominal UVLO turn-on remains 16.63 V; OVP cutoff is now 33.99 V.\nNominal recovery from OVP is 31.78 V. Design input: 24 V nominal;\n18-30 V continuous candidate range, not the former 18-36 V assumption.\nR305=5.1k and MODE latch-off are unchanged. Validate surge let-through\nand all tolerance/temperature corners before hardware release."
 		(exclude_from_sim no)
 		(at 154.94 68.58 0)
@@
 			)
 		)
-		(property "Value" "16k"
+		(property "Value" "14.3k"
 			(at 36.83 113.03 0)
 			(show_name no)
@@
 			)
 		)
-		(property "Datasheet" ""
+		(property "Datasheet" "https://www.yageogroup.com/component-documentation/download/specsheet/RT0402BRD0714K3L"
 			(at 36.83 110.49 0)
 			(hide yes)
@@
 			)
 		)
-		(property "Description" "Chip resistor, 16k Ohm, 1%, 0402; middle UVLO/OVP divider section"
+		(property "Description" "Precision thin-film resistor 14.3k, 0.1%, 25ppm/K, 0402; input UVLO/OVP divider"
 			(at 36.83 110.49 0)
 			(hide yes)
@@
 			)
 		)
-		(property "MPN" "RC0402FR-0716KL"
+		(property "MPN" "RT0402BRD0714K3L"
 			(at 36.83 110.49 0)
 			(hide yes)
@@
 			)
 		)
-		(property "Value" "12k"
+		(property "Value" "13.7k"
 			(at 25.4 113.03 0)
 			(show_name no)
@@
 			)
 		)
-		(property "Datasheet" ""
+		(property "Datasheet" "https://www.yageogroup.com/component-documentation/download/specsheet/RT0402BRD0713K7L"
 			(at 24.13 110.49 0)
 			(hide yes)
@@
 			)
 		)
-		(property "Description" "Chip resistor, 12k Ohm, 1%, 0402; bottom UVLO/OVP divider section"
+		(property "Description" "Precision thin-film resistor 13.7k, 0.1%, 25ppm/K, 0402; input UVLO/OVP divider"
 			(at 24.13 110.49 0)
 			(hide yes)
@@
 			)
 		)
-		(property "MPN" "RC0402FR-0712KL"
+		(property "MPN" "RT0402BRD0713K7L"
 			(at 24.13 110.49 0)
 			(hide yes)
