File: hardware/MIRA_Power/3500_MONITOR_INPUT_AON_USB_SYS.kicad_sch (KiCad schematic)
At the start: 36 parts, among them U3501 INA293A1IDBVR, U3502 INA301A1IDGKR, U3503 INA301A1IDGKR, U3504 INA301A1IDGKR

Commit message: Protect unpowered signal domains and qualify local supplies; retain startup and fault interlocks
MIRA-Startup-Patch: 7ffae17756ebcf923eff1212bb1aade8fbdfae03a9ca8ecebc69d3da3d3b4ba2
Connections:
- net MON_V_INPUT: no longer D3501.3 (K1/A2)
- net MON_V_SYS: no longer D3504.3 (K1/A2)
- net MON_V_USB: no longer D3503.3 (K1/A2)
- new net MON_V_INPUT_SAFE: D3501.3 (K1/A2)
- new net MON_V_SYS_SAFE: D3504.3 (K1/A2)
- new net MON_V_USB_SAFE: D3503.3 (K1/A2)
Changed lines of the file:
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@@
 	(wire
 		(pts
-			(xy 48.26 78.74) (xy 38.1 78.74)
-		)
-		(stroke
-			(width 0)
-			(type default)
-		)
-	)
-	(wire
-		(pts
 			(xy 48.26 73.66) (xy 38.1 73.66)
 		)
@@
 	(wire
 		(pts
-			(xy 110.49 177.8) (xy 110.49 168.91)
-		)
-		(stroke
-			(width 0)
-			(type default)
-		)
-	)
-	(wire
-		(pts
 			(xy 88.9 95.25) (xy 88.9 97.79)
 		)
@@
 	(wire
 		(pts
-			(xy 48.26 86.36) (xy 48.26 78.74)
-		)
-		(stroke
-			(width 0)
-			(type default)
-		)
-	)
-	(wire
-		(pts
 			(xy 100.33 168.91) (xy 88.9 168.91)
 		)
@@
 	(wire
 		(pts
-			(xy 46.99 177.8) (xy 46.99 168.91)
-		)
-		(stroke
-			(width 0)
-			(type default)
-		)
-	)
-	(wire
-		(pts
 			(xy 128.27 162.56) (xy 128.27 163.83)
 		)
@@
 		)
 	)
+(global_label "MON_V_INPUT_SAFE" (shape input) (at 48.26 86.36 180) (effects (font (size 0.8 0.8)) (justify right)))
+(global_label "MON_V_SYS_SAFE" (shape input) (at 110.49 177.8 180) (effects (font (size 0.8 0.8)) (justify right)))
+(global_label "MON_V_USB_SAFE" (shape input) (at 46.99 177.8 180) (effects (font (size 0.8 0.8)) (justify right)))
 )
