File: hardware/MIRA_Power/3600_MONITOR_FPGA_ANA_AFE.kicad_sch (KiCad schematic)
At the start: 27 parts, among them U3601 INA301A1IDGKR, U3602 INA301A1IDGKR, U3603 INA301A1IDGKR

Commit message: Protect unpowered signal domains and qualify local supplies; retain startup and fault interlocks
MIRA-Startup-Patch: 7ffae17756ebcf923eff1212bb1aade8fbdfae03a9ca8ecebc69d3da3d3b4ba2
Connections:
- net MON_V_ANA6: no longer D3602.3 (K1/A2)
- net MON_V_FPGA: no longer D3601.3 (K1/A2)
- net MON_V_P15: no longer D3603.3 (K1/A2)
- new net MON_V_ANA6_SAFE: D3602.3 (K1/A2)
- new net MON_V_FPGA_SAFE: D3601.3 (K1/A2)
- new net MON_V_P15_SAFE: D3603.3 (K1/A2)
Changed lines of the file:
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@@
 	(wire
 		(pts
-			(xy 109.22 179.07) (xy 109.22 170.18)
-		)
-		(stroke
-			(width 0)
-			(type default)
-		)
-	)
-	(wire
-		(pts
 			(xy 53.34 184.15) (xy 54.61 184.15)
 		)
@@
 	(wire
 		(pts
-			(xy 45.72 179.07) (xy 45.72 170.18)
-		)
-		(stroke
-			(width 0)
-			(type default)
-		)
-	)
-	(wire
-		(pts
 			(xy 63.5 52.07) (xy 74.93 52.07)
 		)
@@
 	(wire
 		(pts
-			(xy 45.72 93.98) (xy 45.72 85.09)
-		)
-		(stroke
-			(width 0)
-			(type default)
-		)
-	)
-	(wire
-		(pts
 			(xy 127 137.16) (xy 138.43 137.16)
 		)
@@
 		)
 	)
+(global_label "MON_V_ANA6_SAFE" (shape input) (at 45.72 179.07 180) (effects (font (size 0.8 0.8)) (justify right)))
+(global_label "MON_V_FPGA_SAFE" (shape input) (at 45.72 93.98 180) (effects (font (size 0.8 0.8)) (justify right)))
+(global_label "MON_V_P15_SAFE" (shape input) (at 109.22 179.07 180) (effects (font (size 0.8 0.8)) (justify right)))
 )
