File: hardware/MIRA_Power/MIRA_Power.kicad_sch (KiCad schematic)
At the start: 0 parts

Commit message: Add high-load schematic candidate with CORE sense and revised N15 supply
Other:
- added sheet POWER_CONTROL_INTERFACE (4900_POWER_CONTROL_INTERFACE.kicad_sch)
- note added: "ERC source declarations: verified paths after inductors / current shunts."

Commit message: Protect unpowered signal domains and qualify local supplies; retain startup and fault interlocks
MIRA-Startup-Patch: 7ffae17756ebcf923eff1212bb1aade8fbdfae03a9ca8ecebc69d3da3d3b4ba2
Other:
- added sheet 5200_PM_STARTUP_QUALIFIER (5200_PM_STARTUP_QUALIFIER.kicad_sch)
- added sheet 5300_PM_STARTUP_OUTPUTS (5300_PM_STARTUP_OUTPUTS.kicad_sch)
- added sheet 5400_HOST_LINK_WATCHDOG (5400_HOST_LINK_WATCHDOG.kicad_sch)
- added sheet 5500_AON_HOST_INPUT_ISOLATION (5500_AON_HOST_INPUT_ISOLATION.kicad_sch)
- added sheet 5600_AON_ANALOG_INPUT_ISOLATION (5600_AON_ANALOG_INPUT_ISOLATION.kicad_sch)
- added sheet 5700_AON_ANALOG_INPUT_ISOLATION (5700_AON_ANALOG_INPUT_ISOLATION.kicad_sch)
- added sheet 5800_VIN_REFERENCED_ENABLES (5800_VIN_REFERENCED_ENABLES.kicad_sch)
- added sheet 5900_VIN_REFERENCED_ENABLES (5900_VIN_REFERENCED_ENABLES.kicad_sch)
- added sheet 6000_FPGA_AUX_IO_INTERLOCK (6000_FPGA_AUX_IO_INTERLOCK.kicad_sch)
- added sheet 6100_AON_MONITOR_ENABLE_BUFFER (6100_AON_MONITOR_ENABLE_BUFFER.kicad_sch)
- note added: "MIRA Power / native sheet navigation / signal remediation"
- note removed: "+24V_RAW"
- note removed: "+24V_RAW and +24V_FUSED mark powered input nodes. The GND marker establishes the common reference. Physical sources are on POWER_INPUT."
- note removed: "24 V supply infrastructure for the memristor platform."
- note removed: "ANA6 / ANA5 / ANA3V3 / +/-15 V"
- note removed: "ANA6 feeds the low-noise ANA5 and ANA3V3 branches. P15 and N15 supply the bipolar analog front end and the programming switches. Keeping these domains separately controlled lets the power manager qualify readiness before matrix operation."
- note removed: "Analog and AFE"
- note removed: "Analog and AFE rails"
- note removed: "Block descriptions"
- note removed: "Digital and memory"
- note removed: "Digital and memory rails"
- note removed: "ERC source declarations: verified paths after inductors / current shunts."
- note removed: "External 24 V input"
- note removed: "FPGA / SYS / DDR / PHY"
- note removed: "Groups denote separate rails. Open POWER_SYSTEM for their connections."
- note removed: "MIRA / E4 connection diagram"
- note removed: "MIRA power subsystem overview"
- note removed: "POWER_SYSTEM contains the protected 24 V input, the primary and secondary supply trees, programming switches, power control and rail monitoring. The STM32G0B1 stages startup; hardware permits can remove power independently of telemetry polling."
- note removed: "Positive and negative programming paths use the P15/N15 supplies. MATRIX_PERMIT qualifies operation; the programming interface returns PROG_V_P15 to the power manager. Switch gating and output feedback are detailed on PROGRAM_SWITCHES."
- note removed: "Power source assertions"
- note removed: "Power system"
- note removed: "Programming drive"
- note removed: "Programming drive / control / monitoring"
- note removed: "Protected input / primary and secondary rails"
- note removed: "SHEET GUIDE / MIRA"
- note removed: "Switched programming voltages"
- note removed: "The FPGA intermediate supply feeds core, auxiliary, I/O, DDR and PHY rails. SYS3V3 supports the host-facing power-control interface. These supply domains support matrix timing, data capture, memory and communications in the MIRA platform."
- note removed: "The native hierarchy on this root contains one child: POWER_SYSTEM."
- note removed: "The three PWR_FLAG symbols declare +24V_RAW, +24V_FUSED and GND as powered nodes for electrical-rule checking. These virtual markers support ERC; the physical connector, fuse and input protection are inside POWER_INPUT."
- note removed: "Virtual ERC markers"
- company: MIRA -> (none)
- title: MIRA -> MIRA Power - sheet navigation
